Commit message: Minor fixes to motoman sia10d and robotiq s-model urdfs.
git-svn-id: http://swri-ros-pkg.googlecode.com/svn/trunk@122 076cdf4d-ed99-c8c1-5d01-9bc0d27e81bd

File: industrial/motoman/cfg/sia10d_mesh.xacro (robot description, xacro)
@@ -2,4 +2,4 @@
 <robot name="sia10d_mesh" xmlns:xacro="http://ros.org/wiki/xacro">
 	<include filename="$(find motoman)/cfg/sia10d_mesh_macro.xacro" />
-	<xacro:sia20d_mesh prefix=""/>
+	<xacro:sia10d_mesh prefix=""/>
 </robot>

File: industrial/motoman/cfg/sia10d_mesh_macro.xacro (robot description, xacro)
@@ -1,4 +1,4 @@
 <robot xmlns:xacro="http://ros.org/wiki/xacro">
-	<xacro:macro name="sia20d_mesh" params="prefix">
+	<xacro:macro name="sia10d_mesh" params="prefix">
 		<!-- link list -->
 		<link name="${prefix}base_link">

File: industrial/robotiq/cfg/s-model_mesh_macro.xacro (robot description, xacro)
@@ -57,5 +57,5 @@
 			<collision>
 				<geometry>
-					<mesh filename="package://robotiq/meshes/s-model/collision/GRIPPER_FINGER_3.stl" />
+					<mesh filename="package://robotiq/meshes/s-model/collision/GRIPPER_OPEN_FINGER_3.stl" />
 				</geometry>
 				<material name="yellow"/>
