Commit message: Minor changes in order to get trajectory downloading to work (still isn't working though).  Cleaned up logging, removed duplicate, unneeded messages.  A key change was made to TrajectoryJob class, removing the JointTraj from the class.  This seems to have fixed a controller crash, though I'm not sure why.  I have a feeling there is a memory issue with the controller and having a large class creates problems.  It is also possible that I am dynamically allocating memory somewhere (maybe where I use static const variables to initialize array sizes), which I have avoided doing.
git-svn-id: http://swri-ros-pkg.googlecode.com/svn/trunk@301 076cdf4d-ed99-c8c1-5d01-9bc0d27e81bd

File: industrial/motoman/cfg/sia20d_mesh.xacro (robot description, xacro)
@@ -2,4 +2,4 @@
 <robot name="SIA20D_Mesh" xmlns:xacro="http://ros.org/wiki/xacro">
 	<include filename="$(find motoman)/cfg/sia20d_mesh_macro.xacro" />
-	<xacro:sia20d_mesh/>
+	<xacro:sia20d_mesh prefix=""/>
 </robot>

File: industrial/motoman/cfg/sia20d_mesh_macro.xacro (robot description, xacro)
@@ -1,6 +1,6 @@
 <robot xmlns:xacro="http://ros.org/wiki/xacro">
-	<xacro:macro name="sia20d_mesh">
+	<xacro:macro name="sia20d_mesh" params="prefix">
 		<!-- link list -->
-		<link name="base_link">
+		<link name="${prefix}base_link">
 			<visual>
 				<geometry>
@@ -20,6 +20,7 @@
 			</collision>
 		</link>
-		<link name="link_s">
+		<link name="${prefix}link_s">
 			<visual>
+				<origin rpy="0 0 3.1416" xyz="0 0 0"/>
 				<geometry>
 					<mesh filename="package://motoman/meshes/sia20d/visual/MOTOMAN_AXIS_S.stl"/>
@@ -30,4 +31,5 @@
 			</visual>
 			<collision>
+				<origin rpy="0 0 3.1416" xyz="0 0 0"/>
 				<geometry>
 					<mesh filename="package://motoman/meshes/sia20d/collision/MOTOMAN_AXIS_S.stl" />
@@ -36,6 +38,7 @@
 			</collision>
 		</link>
-		<link name="link_l">
+		<link name="${prefix}link_l">
 			<visual>
+				<origin rpy="1.57 3.1416 3.1416" xyz="0 0 0"/>
 				<geometry>
 					<mesh filename="package://motoman/meshes/sia20d/visual/MOTOMAN_AXIS_L.stl"/>
@@ -44,4 +47,5 @@
 			</visual>
 			<collision>
+				<origin rpy="1.57 3.1416 3.1416" xyz="0 0 0"/>
 				<geometry>
 					<mesh filename="package://motoman/meshes/sia20d/collision/MOTOMAN_AXIS_L.stl"/>
@@ -50,6 +54,7 @@
 			</collision>
 		</link>
-		<link name="link_e">
+		<link name="${prefix}link_e">
 			<visual>
+				<origin rpy="0 0 0" xyz="0 0 0"/>
 				<geometry>
 					<mesh filename="package://motoman/meshes/sia20d/visual/MOTOMAN_AXIS_E.stl"/>
@@ -58,4 +63,5 @@
 			</visual>
 			<collision>
+				<origin rpy="0 0 0" xyz="0 0 0"/>
 				<geometry>
 					<mesh filename="package://motoman/meshes/sia20d/collision/MOTOMAN_AXIS_E.stl"/>
@@ -64,6 +70,7 @@
 			</collision>
 		</link>
-		<link name="link_u">
+		<link name="${prefix}link_u">
 			<visual>
+				<origin rpy="1.57 -3.1415 3.1416" xyz="0 0 0"/>
 				<geometry>
 					<mesh filename="package://motoman/meshes/sia20d/visual/MOTOMAN_AXIS_U.stl"/>
@@ -72,4 +79,5 @@
 			</visual>
 			<collision>
+				<origin rpy="1.57 -3.1415 3.1416" xyz="0 0 0"/>
 				<geometry>
 					<mesh filename="package://motoman/meshes/sia20d/collision/MOTOMAN_AXIS_U.stl"/>
@@ -78,6 +86,7 @@
 			</collision>
 		</link>
-		<link name="link_r">
+		<link name="${prefix}link_r">
 			<visual>
+				<origin rpy="0 0 0" xyz="0 0 0"/>
 				<geometry>
 					<mesh filename="package://motoman/meshes/sia20d/visual/MOTOMAN_AXIS_R.stl"/>
@@ -86,4 +95,5 @@
 			</visual>
 			<collision>
+				<origin rpy="0 0 0" xyz="0 0 0"/>
 				<geometry>
 					<mesh filename="package://motoman/meshes/sia20d/collision/MOTOMAN_AXIS_R.stl"/>
@@ -92,6 +102,7 @@
 			</collision>
 		</link>
-		<link name="link_b">
+		<link name="${prefix}link_b">
 			<visual>
+				<origin rpy="-1.57 0 0" xyz="0 0 0"/>
 				<geometry>
 					<mesh filename="package://motoman/meshes/sia20d/visual/MOTOMAN_AXIS_B.stl"/>
@@ -100,4 +111,5 @@
 			</visual>
 			<collision>
+				<origin rpy="-1.57 0 0" xyz="0 0 0"/>
 				<geometry>
 					<mesh filename="package://motoman/meshes/sia20d/collision/MOTOMAN_AXIS_B.stl"/>
@@ -106,5 +118,5 @@
 			</collision>
 		</link>
-		<link name="link_t">
+		<link name="${prefix}link_t">
 			<visual>
 				<geometry>
@@ -122,50 +134,50 @@
 		<!-- end of link list -->
 		<!-- joint list -->
-		<joint name="joint_s" type="revolute">
+		<joint name="${prefix}joint_s" type="revolute">
 			<parent link="base_link"/>
 			<child link="link_s"/>
-			<origin xyz="0 0 0.41" rpy="0 0 3.1415"/>
+			<origin xyz="0 0 0.41" rpy="0 0 0"/>
 			<axis xyz="0 0 1" />
-			<limit lower="-3.1416" upper="3.1416" effort="100" velocity="2.66" />
+			<limit lower="-3.1416" upper="3.1416" effort="100" velocity="2.26" />
 		</joint>
-		<joint name="joint_l" type="revolute">
+		<joint name="${prefix}joint_l" type="revolute">
 			<parent link="link_s"/>
 			<child link="link_l"/>
-			<origin xyz="0 0 0" rpy="1.570 3.1416 0"/>
-			<axis xyz="0 0 1" />
-			<limit lower="-1.91" upper="1.91" effort="100" velocity="2.66" />
+			<origin xyz="0 0 0" rpy="0 0 0"/>
+			<axis xyz="0 1 0" />
+			<limit lower="-1.91" upper="1.91" effort="100" velocity="2.26" />
 		</joint>
-		<joint name="joint_e" type="revolute">
+		<joint name="${prefix}joint_e" type="revolute">
 			<parent link="link_l"/>
 			<child link="link_e"/>
-			<origin xyz="0 -0.49 0" rpy="1.570 0 0"/>
+			<origin xyz="0 0 0.49" rpy="0 0 0"/>
 			<axis xyz="0 0 1" />
 			<limit lower="-2.96" upper="2.96" effort="100" velocity="2.96" />
 		</joint>
-		<joint name="joint_u" type="revolute">
+		<joint name="${prefix}joint_u" type="revolute">
 			<parent link="link_e"/>
 			<child link="link_u"/>
-			<origin xyz="0 0 0" rpy="-1.570 0 0"/>
-			<axis xyz="0 0 -1" />
-			<limit lower="-3.1416" upper="3.1416" effort="100" velocity="2.96" />
+			<origin xyz="0 0 0" rpy="0 0 0"/>
+			<axis xyz="0 -1 0" />
+			<limit lower="-2.26" upper="2.26" effort="100" velocity="2.96" />
 		</joint>
-		<joint name="joint_r" type="revolute">
+		<joint name="${prefix}joint_r" type="revolute">
 			<parent link="link_u"/>
 			<child link="link_r"/>
-			<origin xyz="0 -0.420 0" rpy="1.570 0 0"/>
+			<origin xyz="0 0 0.420" rpy="0 0 0"/>
 			<axis xyz="0 0 -1" />
 			<limit lower="-3.1416" upper="3.1416" effort="100" velocity="3.48" />
 		</joint>
-		<joint name="joint_b" type="revolute">
+		<joint name="${prefix}joint_b" type="revolute">
 			<parent link="link_r"/>
 			<child link="link_b"/>
-			<origin xyz="0 0 0" rpy="-1.570 0 0"/>
-			<axis xyz="0 0 -1" />
+			<origin xyz="0 0 0" rpy="0 0 0"/>
+			<axis xyz="0 -1 0" />
 			<limit lower="-1.91" upper="1.91" effort="100" velocity="3.48" />
 		</joint>
-		<joint name="joint_t" type="revolute">
+		<joint name="${prefix}joint_t" type="revolute">
 			<parent link="link_b"/>
 			<child link="link_t"/>
-			<origin xyz="0 -0.18 0" rpy="1.570 0 0"/>
+			<origin xyz="0 0 0.18" rpy="0 0 0"/>
 			<axis xyz="0 0 -1" />
 			<limit lower="-3.1416" upper="3.1416" effort="100" velocity="6.97" />
