Commit message: Added table(s) and kinect sensor to armadillo urdf file.  NOTE: the arm wizard was not rerun to account for the changes.  This may or may not be OK.
git-svn-id: http://swri-ros-pkg.googlecode.com/svn/trunk@124 076cdf4d-ed99-c8c1-5d01-9bc0d27e81bd

File: industrial/armadillo/cfg/armadillo.xacro (robot description, xacro)
@@ -78,4 +78,24 @@
 			</visual>
 		</link>
+    <link name="kinect">
+			<visual>
+				<geometry>
+					<box size="0.36 0.28 0.22"/>
+				</geometry>
+				<material name="">
+					<color rgba="1 0.8 1 1"/>
+				</material>
+			</visual>
+		</link>
+    <link name="tables">
+			<visual>
+				<geometry>
+					<box size="1.10 1.65 0.45"/>
+				</geometry>
+				<material name="">
+					<color rgba="1 0.7 1 1"/>
+				</material>
+			</visual>
+		</link>
 		<joint name="base-pallet" type="fixed">
 			<parent link="base_link"/>
@@ -98,4 +118,14 @@
 			<origin xyz="0 0 -0.11" rpy="0 0 0"/>
 		</joint>
+		<joint name="filter-kinect" type="fixed">
+			<parent link="filter"/>
+			<child link="kinect"/>
+			<origin xyz="0.18 0 0.29" rpy="0 0 0"/>
+		</joint>
+		<joint name="base-tables" type="fixed">
+			<parent link="base_link"/>
+			<child link="tables"/>
+			<origin xyz="0.84 0 0" rpy="0 0 0"/>
+		</joint>
   <!-- end environment list -->
 </robot>

Commit message: Fixed orientation of robotiq hand (it was 180 degrees off).  NOTE: Arm wizard not rerun on new URDF.
git-svn-id: http://swri-ros-pkg.googlecode.com/svn/trunk@129 076cdf4d-ed99-c8c1-5d01-9bc0d27e81bd

File: industrial/armadillo/cfg/armadillo.xacro (robot description, xacro)
@@ -34,5 +34,5 @@
 			<parent link="coupler"/>
 			<child link="palm"/>
-			<origin xyz="0 0.240 0" rpy="-1.570 2.665 0"/>
+			<origin xyz="0 0.240 0" rpy="-1.570 -0.478 0"/>
 		</joint>
   <!-- end of joint list -->

Commit message: Adding table top launch file.
git-svn-id: http://swri-ros-pkg.googlecode.com/svn/trunk@201 076cdf4d-ed99-c8c1-5d01-9bc0d27e81bd

File: industrial/armadillo/cfg/armadillo.xacro (robot description, xacro)
@@ -129,3 +129,63 @@
 		</joint>
   <!-- end environment list -->
+  <!-- kinect -->
+		<joint name="kinect_frame_joint" type="fixed">
+			<parent link="kinect"/>
+			<child link="kinect_frame"/>
+			<origin rpy="0.075 0.351422870712 0.396594014755" xyz="-0.12481258247 0.064659133914 -0.022541275619"/>
+		</joint>
+		<link name="kinect_frame">
+			<visual>
+				<origin rpy="0 0 0" xyz="0 0 0"/>
+				<geometry>
+					<box size="0.064 0.28 0.04"/>
+				</geometry>
+				<material name="silver"/>
+			</visual>
+			<collision>
+				<origin rpy="0 0 0" xyz="0 0 0"/>
+				<geometry>
+					<box size="0.064 0.28 0.04"/>
+				</geometry>
+			</collision>
+		</link>
+		<joint name="kinect_ir_joint" type="fixed">
+			<parent link="kinect_frame"/>
+			<child link="kinect_ir_link"/>
+			<origin rpy="0 0 0" xyz="0 0 0"/>
+		</joint>
+		<link name="kinect_ir_link">
+			<visual>
+				<origin rpy="0 0 0" xyz="0 0 0"/>
+				<geometry>
+					<sphere radius="0.0005"/>
+				</geometry>
+			</visual>
+		</link>
+		<joint name="kinect_ir_optical_frame_joint" type="fixed">
+			<parent link="kinect_ir_link"/>
+			<child link="kinect_ir_optical_frame"/>
+			<origin rpy="-1.57 0 -1.57" xyz="0 0 0"/>
+		</joint>
+		<link name="kinect_ir_optical_frame"/>
+		<joint name="kinect_rgb_joint" type="fixed">
+			<parent link="kinect_ir_link"/>
+			<child link="kinect_rgb_link"/>
+			<origin rpy="0 0 0" xyz="0 -0.03 0"/>
+		</joint>
+		<link name="kinect_rgb_link">
+			<visual>
+				<origin rpy="0 0 0" xyz="0 0 0"/>
+				<geometry>
+					<sphere radius="0.0005"/>
+				</geometry>
+			</visual>
+		</link>
+		<joint name="kinect_rgb_optical_frame_joint" type="fixed">
+			<parent link="kinect_rgb_link"/>
+			<child link="kinect_rgb_optical_frame"/>
+			<origin rpy="-1.57 0 -1.57" xyz="0 0 0"/>
+		</joint>
+		<link name="kinect_rgb_optical_frame"/>
+  <!-- end kinect -->
 </robot>

File: industrial/motoman/cfg/sia10d_mesh_macro.xacro (robot description, xacro)
@@ -1,2 +1,3 @@
+<?xml version="1.0" ?>
 <robot xmlns:xacro="http://ros.org/wiki/xacro">
 	<xacro:macro name="sia10d_mesh" params="prefix">
@@ -38,4 +39,5 @@
 		<link name="${prefix}link_l">
 			<visual>
+				<origin rpy="1.57 3.1416 0" xyz="0 0 0"/>
 				<geometry>
 					<mesh filename="package://motoman/meshes/sia10d/visual/MOTOMAN_AXIS_L.stl"/>
@@ -44,4 +46,5 @@
 			</visual>
 			<collision>
+				<origin rpy="1.57 3.1416 0" xyz="0 0 0"/>
 				<geometry>
 					<mesh filename="package://motoman/meshes/sia10d/collision/MOTOMAN_AXIS_L.stl" />
@@ -52,4 +55,5 @@
 		<link name="${prefix}link_e">
 			<visual>
+				<origin rpy="0 0 3.1415" xyz="0 0 0"/>
 				<geometry>
 					<mesh filename="package://motoman/meshes/sia10d/visual/MOTOMAN_AXIS_E.stl"/>
@@ -58,4 +62,5 @@
 			</visual>
 			<collision>
+				<origin rpy="0 0 3.1415" xyz="0 0 0"/>
 				<geometry>
 					<mesh filename="package://motoman/meshes/sia10d/collision/MOTOMAN_AXIS_E.stl" />
@@ -66,4 +71,5 @@
 		<link name="${prefix}link_u">
 			<visual>
+				<origin rpy="1.57 -3.1415 0" xyz="0 0 0"/>
 				<geometry>
 					<mesh filename="package://motoman/meshes/sia10d/visual/MOTOMAN_AXIS_U.stl"/>
@@ -72,4 +78,5 @@
 			</visual>
 			<collision>
+				<origin rpy="1.57 -3.1415 0" xyz="0 0 0"/>
 				<geometry>
 					<mesh filename="package://motoman/meshes/sia10d/collision/MOTOMAN_AXIS_U.stl" />
@@ -80,4 +87,5 @@
 		<link name="${prefix}link_r">
 			<visual>
+				<origin rpy="0 0 3.1416" xyz="0 0 0"/>
 				<geometry>
 					<mesh filename="package://motoman/meshes/sia10d/visual/MOTOMAN_AXIS_R.stl"/>
@@ -86,4 +94,5 @@
 			</visual>
 			<collision>
+				<origin rpy="0 0 3.1416" xyz="0 0 0"/>
 				<geometry>
 					<mesh filename="package://motoman/meshes/sia10d/collision/MOTOMAN_AXIS_R.stl" />
@@ -94,4 +103,5 @@
 		<link name="${prefix}link_b">
 			<visual>
+				<origin rpy="-1.57 0 3.1416" xyz="0 0 0"/>
 				<geometry>
 					<mesh filename="package://motoman/meshes/sia10d/visual/MOTOMAN_AXIS_B.stl"/>
@@ -100,4 +110,5 @@
 			</visual>
 			<collision>
+				<origin rpy="-1.57 0 3.1416" xyz="0 0 0"/>
 				<geometry>
 					<mesh filename="package://motoman/meshes/sia10d/collision/MOTOMAN_AXIS_B.stl" />
@@ -125,5 +136,5 @@
 			<parent link="base_link"/>
 			<child link="link_s"/>
-			<origin xyz="0 0 0.36" rpy="0 0 3.1415"/>
+			<origin xyz="0 0 0.36" rpy="0 0 0"/>
 			<axis xyz="0 0 1" />
 			<limit lower="-3.1416" upper="3.1416" effort="100" velocity="2.96" />
@@ -132,6 +143,6 @@
 			<parent link="link_s"/>
 			<child link="link_l"/>
-			<origin xyz="0 0 0" rpy="1.570 3.1416 0"/>
-			<axis xyz="0 0 1" />
+			<origin xyz="0 0 0" rpy="0 0 0"/>
+			<axis xyz="0 1 0" />
 			<limit lower="-1.91" upper="1.91" effort="100" velocity="2.96" />
 		</joint>
@@ -139,5 +150,5 @@
 			<parent link="link_l"/>
 			<child link="link_e"/>
-			<origin xyz="0 -0.36 0" rpy="1.570 0 0"/>
+			<origin xyz="0 0 0.36" rpy="0 0 0"/>
 			<axis xyz="0 0 1" />
 			<limit lower="-2.96" upper="2.96" effort="100" velocity="2.96" />
@@ -146,6 +157,6 @@
 			<parent link="link_e"/>
 			<child link="link_u"/>
-			<origin xyz="0 0 0" rpy="-1.570 0 0"/>
-			<axis xyz="0 0 -1" />
+			<origin xyz="0 0 0" rpy="0 0 0"/>
+			<axis xyz="0 -1 0" />
 			<limit lower="-2.35" upper="2.35" effort="100" velocity="2.96" />
 		</joint>
@@ -153,5 +164,5 @@
 			<parent link="link_u"/>
 			<child link="link_r"/>
-			<origin xyz="0 -0.360 0" rpy="1.570 0 0"/>
+			<origin xyz="0 0 0.360" rpy="0 0 0"/>
 			<axis xyz="0 0 -1" />
 			<limit lower="-3.1416" upper="3.1416" effort="100" velocity="3.48" />
@@ -160,6 +171,6 @@
 			<parent link="link_r"/>
 			<child link="link_b"/>
-			<origin xyz="0 0 0" rpy="-1.570 0 0"/>
-			<axis xyz="0 0 -1" />
+			<origin xyz="0 0 0" rpy="0 0 0"/>
+			<axis xyz="0 -1 0" />
 			<limit lower="-1.91" upper="1.91" effort="100" velocity="3.48" />
 		</joint>
@@ -167,5 +178,5 @@
 			<parent link="link_b"/>
 			<child link="link_t"/>
-			<origin xyz="0 -0.155 0" rpy="1.570 0 0"/>
+			<origin xyz="0 0 0.155" rpy="0 0 0"/>
 			<axis xyz="0 0 -1" />
 			<limit lower="-3.1416" upper="3.1416" effort="100" velocity="6.97" />
