Commit message: Fixed urdf to match physical robot.
git-svn-id: http://swri-ros-pkg.googlecode.com/svn/trunk@217 076cdf4d-ed99-c8c1-5d01-9bc0d27e81bd

File: adept/adept_common/urdf/Adept_Viper_s650.urdf (robot description, URDF)
Before this commit: robot ADEPT_VIPER_S650, 7 links, 6 joints
Joints:
- joint joint_3: origin xyz=0 0 0.270 -> xyz=0.270 0 0
- joint joint_4: axis 1 0 0 -> 0 0 1; origin xyz=0.295 0 0.090 -> xyz=-0.090 0 0.295
- joint joint_6: axis 1 0 0 -> 0 0 1; origin xyz=0.08 0 0 -> xyz=0.0 0 0.08

Commit message: Added joint velocity limits to the URDF.
git-svn-id: http://swri-ros-pkg.googlecode.com/svn/trunk@223 076cdf4d-ed99-c8c1-5d01-9bc0d27e81bd

File: adept/adept_common/urdf/Adept_Viper_s650.urdf (robot description, URDF)
Before this commit: robot ADEPT_VIPER_S650, 7 links, 6 joints
Joints:
- joint joint_1: limit lower=-2.9670 upper=2.9670 effort=100 velocity=1.0 -> lower=-2.9670 upper=2.9670 effort=100 velocity=5.72468
- joint joint_2: limit lower=-3.31613 upper=0.7854 effort=100 velocity=1.0 -> lower=-3.31613 upper=0.7854 effort=100 velocity=5.235
- joint joint_3: limit lower=-0.50615 upper=4.468053 effort=100 velocity=1.0 -> lower=-0.50615 upper=4.468053 effort=100 velocity=6.544
- joint joint_4: limit lower=-3.31613 upper=3.316133 effort=100 velocity=1.0 -> lower=-3.31613 upper=3.316133 effort=100 velocity=6.544
- joint joint_5: limit lower=-2.0944 upper=2.0944 effort=100 velocity=1.0 -> lower=-2.0944 upper=2.0944 effort=100 velocity=6.544
- joint joint_6: limit lower=-3.1416 upper=3.1416 effort=100 velocity=1.0 -> lower=-3.1416 upper=3.1416 effort=100 velocity=10.47
