Commit message: Added collision model for power supply.  The visual model does not appear to be used as a collision model in the absence of a specified model.
git-svn-id: http://swri-ros-pkg.googlecode.com/svn/trunk@309 076cdf4d-ed99-c8c1-5d01-9bc0d27e81bd

File: industrial/longhorn/cfg/longhorn.xacro (robot description, xacro)
@@ -95,4 +95,12 @@
 				</material>
 			</visual>
+			<collision>
+				<geometry>
+					<box size="0.400 0.250 0.115"/>
+				</geometry>
+				<material name="">
+					<color rgba="1 0.2 1 0.1"/>
+				</material>
+			</collision>
 		</link>
 		<link name="kinect_keepout">
