Commit message: Actual robot/gripper integrated to demo
git-svn-id: http://swri-ros-pkg.googlecode.com/svn/trunk@514 076cdf4d-ed99-c8c1-5d01-9bc0d27e81bd

File: freetail/freetail_config/urdf/freetail_vacuum_gripper_conf.urdf (robot description, URDF)
Before this commit: robot freetail, 22 links, 21 joints
Links:
- link palm: geometry collision box size=0.040 0.080 0.0946; visual box size=0.040 0.080 0.0946
Joints:
- joint coupler-hand: origin xyz=0 0.196 0.019 rpy=-1.570 0 0 -> xyz=-0.013 0.182 -0.013 rpy=-1.570 -2.36 0
- joint tool-coupler: origin xyz=0 0 0 rpy=1.570 0 0 -> xyz=0 0 0 rpy=1.570 0 1.57

File: freetail/freetail_config/urdf/freetail_vacuum_gripper_conf.xacro (robot description, xacro)
@@ -29,10 +29,10 @@
 		<parent link="link_t"/>
 		<child link="coupler"/>
-		<origin xyz="0 0 0" rpy="1.570 0 0"/>
+		<origin xyz="0 0 0" rpy="1.570 0 1.57"/>
 	</joint>
 	<joint name="coupler-hand" type="fixed">
 		<parent link="coupler"/>
 		<child link="palm"/>
-		<origin xyz="0 0.196 0.019" rpy="-1.570 0 0"/>
+		<origin xyz="-0.013 0.182 -0.013" rpy="-1.570 -2.36 0"/>
 	</joint>
   <!-- environment list -->

File: freetail/freetail_config/urdf/vacuum_gripper.xacro (robot description, xacro)
@@ -4,7 +4,7 @@
 		<link name="${prefix}palm">
 			<visual>
-				<origin xyz="0 0.019 -0.0543" rpy="0 0 0"/>
+				<origin xyz="0 0.019 -0.0473" rpy="0 0 0"/>
 				<geometry>
-					<box size="0.040 0.080 0.1086"/>
+					<box size="0.040 0.080 0.0946"/>
 				</geometry>
 				<material name="another_blue1">
@@ -13,7 +13,7 @@
 			</visual>
 			<collision>
-				<origin xyz="0 0.019 -0.0543" rpy="0 0 0"/>
+				<origin xyz="0 0.019 -0.0473" rpy="0 0 0"/>
 				<geometry>
-					<box size="0.040 0.080 0.1086"/>
+					<box size="0.040 0.080 0.0946"/>
 				</geometry>
 				<material name="another_blue2">

Commit message: Updated Demo Instructions and made small modifications to TCP placement in urdf
git-svn-id: http://swri-ros-pkg.googlecode.com/svn/trunk@515 076cdf4d-ed99-c8c1-5d01-9bc0d27e81bd

File: freetail/freetail_config/urdf/freetail_vacuum_gripper_conf.urdf (robot description, URDF)
Before this commit: robot freetail, 22 links, 21 joints
Links:
- link palm: geometry collision box size=0.044 0.088 0.0946; visual box size=0.044 0.088 0.0946
Joints:
- joint coupler-hand: origin xyz=-0.013 0.182 -0.013 rpy=-1.570 -2.36 0 -> xyz=0 0.182 0.038 rpy=-1.570 0 0
- joint tool-coupler: origin xyz=0 0 0 rpy=1.570 0 1.57 -> xyz=0 0 0 rpy=1.570 0 -0.785

File: freetail/freetail_config/urdf/freetail_vacuum_gripper_conf.xacro (robot description, xacro)
@@ -29,10 +29,10 @@
 		<parent link="link_t"/>
 		<child link="coupler"/>
-		<origin xyz="0 0 0" rpy="1.570 0 1.57"/>
+		<origin xyz="0 0 0" rpy="1.570 0 -0.785"/>
 	</joint>
 	<joint name="coupler-hand" type="fixed">
 		<parent link="coupler"/>
 		<child link="palm"/>
-		<origin xyz="-0.013 0.182 -0.013" rpy="-1.570 -2.36 0"/>
+		<origin xyz="0 0.182 0.036" rpy="-1.570 0 0"/>
 	</joint>
   <!-- environment list -->

File: freetail/freetail_config/urdf/vacuum_gripper.xacro (robot description, xacro)
@@ -4,7 +4,7 @@
 		<link name="${prefix}palm">
 			<visual>
-				<origin xyz="0 0.019 -0.0473" rpy="0 0 0"/>
+				<origin xyz="0 0.036 -0.0473" rpy="0 0 0"/>
 				<geometry>
-					<box size="0.040 0.080 0.0946"/>
+					<box size="0.044 0.088 0.0946"/>
 				</geometry>
 				<material name="another_blue1">
@@ -13,7 +13,7 @@
 			</visual>
 			<collision>
-				<origin xyz="0 0.019 -0.0473" rpy="0 0 0"/>
+				<origin xyz="0 0.036 -0.0473" rpy="0 0 0"/>
 				<geometry>
-					<box size="0.040 0.080 0.0946"/>
+					<box size="0.044 0.088 0.0946"/>
 				</geometry>
 				<material name="another_blue2">
