Commit message: with corrected link 1 visual mesh
git-svn-id: http://swri-ros-pkg.googlecode.com/svn/trunk@523 076cdf4d-ed99-c8c1-5d01-9bc0d27e81bd

File: abb/abb_common/urdf/irb_2400.urdf (robot description, URDF)
Before this commit: robot irb_2400, 8 links, 7 joints
Links:
- link base_link: geometry collision mesh filename=package://abb_common/meshes/irb_2400/collision/base_link.STL; visual mesh filename=package://abb_common/meshes/irb_2400/visual/base_link.STL
- link link_1: geometry collision mesh filename=package://abb_common/meshes/irb_2400/collision/link_1.STL; visual mesh filename=package://abb_common/meshes/irb_2400/visual/link_1.STL
- link link_2: geometry collision mesh filename=package://abb_common/meshes/irb_2400/collision/link_2_whole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; visual mesh filename=package://abb_common/meshes/irb_2400/visual/link_2.STL
- link link_3: geometry collision mesh filename=package://abb_common/meshes/irb_2400/collision/link_3.STL; visual mesh filename=package://abb_common/meshes/irb_2400/visual/link_3.STL
- link link_4: geometry collision mesh filename=package://abb_common/meshes/irb_2400/collision/link_4.STL; visual mesh filename=package://abb_common/meshes/irb_2400/visual/link_4.STL
- link link_5: geometry collision mesh filename=package://abb_common/meshes/irb_2400/collision/link_5.STL; visual mesh filename=package://abb_common/meshes/irb_2400/visual/link_5.STL
- link link_6: geometry collision mesh filename=package://abb_common/meshes/irb_2400/collision/link_6.STL; visual mesh filename=package://abb_common/meshes/irb_2400/visual/link_6.STL

Commit message: Updated after following changes to irb_2400_macro.xacro: Changed the joint axis orientation on joints 1, 3, and 6, from negatives to positive to match the actual robot joint motion. Also commented out the safety contoller parameters for now (helps with the arm navigation wizard to have this commented out).
git-svn-id: http://swri-ros-pkg.googlecode.com/svn/trunk@525 076cdf4d-ed99-c8c1-5d01-9bc0d27e81bd

File: abb/abb_common/urdf/irb_2400.urdf (robot description, URDF)
Before this commit: robot irb_2400, 8 links, 7 joints
Joints:
- joint joint_1: axis 0 0 -1 -> 0 0 1
- joint joint_2: axis 2.6688E-16 1 0 -> 0 1 0
- joint joint_3: axis 0 -1 0 -> 0 1 0
- joint joint_6: axis -1 0 0 -> 1 0 0
