Commit message: Made IRB-120 orange.

File: abb/abb_common/urdf/irb_120_macro.xacro (robot description, xacro)
@@ -8,7 +8,9 @@
 			</geometry>
 			<origin rpy="0 0 0" xyz="0.04203954 -0.07963916 8.0162399451e-05"/>
-			<material name="IRB120_Base_rev0:11_color">
-				<color rgba="0.752941 0.752941 0.752941 1"/>
-			</material>
+      			<material
+        			name="abb_orange">
+        			<color
+          			rgba="1 0.43 0 1" />
+      			</material>
 		</visual>
 		<inertial>
@@ -30,7 +32,9 @@
 			</geometry>
 			<origin rpy="0 0 0" xyz="0 -0.17649952 0"/>
-			<material name="IRB120_Link1_rev0:11_color">
-				<color rgba="0.752941 0.752941 0.752941 1"/>
-			</material>
+      			<material
+        			name="abb_orange">
+        			<color
+          			rgba="1 0.43 0 1" />
+      			</material>
 		</visual>
 		<inertial>
@@ -52,7 +56,9 @@
 			</geometry>
             <origin rpy="0 0 0" xyz="1.54358428872e-06 0.269999754796 0.115499748015"/>
-			<material name="IRB120_Link2_rev0:11_color">
-				<color rgba="0.752941 0.752941 0.752941 1"/>
-			</material>
+      			<material
+        			name="abb_orange">
+        			<color
+          			rgba="1 0.43 0 1" />
+      			</material>
 		</visual>
 		<inertial>
@@ -74,7 +80,9 @@
 			</geometry>
             <origin rpy="0 0 0" xyz="0.071952848745 -0.0661526901756 0.0589997805382"/>
-			<material name="IRB120_Link3_rev0:11_color">
-				<color rgba="0.752941 0.752941 0.752941 1"/>
-			</material>
+      			<material
+        			name="abb_orange">
+        			<color
+          			rgba="1 0.43 0 1" />
+      			</material>
 		</visual>
 		<inertial>
@@ -96,7 +104,9 @@
 			</geometry>
 			<origin rpy="0 0 0" xyz="500.302187012 0.00151561224702 -0.000313229561613"/>
-			<material name="IRB120_Link4_rev0:11_color">
-				<color rgba="0.752941 0.752941 0.752941 1"/>
-			</material>
+      			<material
+        			name="abb_orange">
+        			<color
+          			rgba="1 0.43 0 1" />
+      			</material>
 		</visual>
 		<inertial>
@@ -118,7 +128,9 @@
 			</geometry>
 			<origin rpy="0 0 0" xyz="-0.301998488439 -0.629998750685 -0.0619993114233"/>
-			<material name="IRB120_Link5_rev0:11_color">
-				<color rgba="0.752941 0.752941 0.752941 1"/>
-			</material>
+      			<material
+        			name="abb_orange">
+        			<color
+          			rgba="1 0.43 0 1" />
+      			</material>
 		</visual>
 		<inertial>
@@ -140,7 +152,9 @@
 			</geometry>
 			<origin rpy="0 0 0" xyz="-2.74896335695e-07 -8.57788299224e-07 -0.0130000906507"/>
-			<material name="IRB120_Link6_rev0:11_color">
-				<color rgba="0.752941 0.752941 0.752941 1"/>
-			</material>
+      			<material
+        			name="abb_orange">
+        			<color
+          			rgba="1 0.43 0 1" />
+      			</material>
 		</visual>
 		<inertial>

Commit message: Updated joint limits for irb 120.

File: abb/abb_common/urdf/irb_120_macro.xacro (robot description, xacro)
@@ -187,5 +187,5 @@
 		<parent link="${prefix}link_2"/>
 		<child link="${prefix}link_3"/>
-		<limit effort="300" lower="-1.92" upper="1.22" velocity="4.36"/>
+		<limit effort="300" lower="-1.575" upper="1.23" velocity="4.36"/>
 		<axis xyz="0 0 -1"/>
 		<origin rpy="3.14159265359 0 3.14159265359" xyz="0 0.270000153642 0.108"/>
@@ -194,5 +194,5 @@
 		<parent link="${prefix}link_3"/>
 		<child link="${prefix}link_4"/>
-		<limit effort="300" lower="-2.79" upper="2.79" velocity="5.58"/>
+		<limit effort="300" lower="-2.80" upper="2.80" velocity="5.58"/>
 		<axis xyz="1 0 0"/>
 		<origin rpy="0 0 0" xyz="-500.000188071 0.0701403024607 0.060593734446"/>
@@ -201,5 +201,5 @@
 		<parent link="${prefix}link_4"/>
 		<child link="${prefix}link_5"/>
-		<limit effort="300" lower="-2.09" upper="2.09" velocity="5.58"/>
+		<limit effort="300" lower="-2.10" upper="2.10" velocity="5.58"/>
 		<axis xyz="0 0 -1"/>
 		<origin rpy="0 0 0" xyz="500.302186066 0.00151566707848 0.0616850168905"/>
@@ -208,5 +208,5 @@
 		<parent link="${prefix}link_5"/>
 		<child link="${prefix}link_6"/>
-		<limit effort="300" lower="-6.98" upper="6.98" velocity="7.33"/>
+		<limit effort="300" lower="-6.985" upper="6.985" velocity="7.33"/>
 		<axis xyz="0 0 1"/>
 		<origin rpy="-1.5707961734 0 -1.57079621992" xyz="0.072000865279 0 -0.0620001796247"/>

Commit message: Removes strange 500 inch offset in link 4.
Link 4's origin was translated 500 inches in the x direction for
some reason. I removed the 500 inch translations wherever they
existed and have examined the resulting model in rviz; it is correct.

File: abb/abb_common/urdf/irb_120_macro.xacro (robot description, xacro)
@@ -103,5 +103,5 @@
 				<mesh filename="package://abb_common/meshes/irb_120/visual/link_4.stl" scale="0.0254 0.0254 0.0254"/>
 			</geometry>
-			<origin rpy="0 0 0" xyz="500.302187012 0.00151561224702 -0.000313229561613"/>
+			<origin rpy="0 0 0" xyz="0.302187012 0.00151561224702 -0.000313229561613"/>
       			<material
         			name="abb_orange">
@@ -113,5 +113,5 @@
 			<mass value="1.32790527095"/>
 			<inertia ixx="0.00284579825479" ixy="1.64819596414e-05" ixz="-2.12443634431e-05" iyy="0.0052535657425" iyz="1.31403377384e-05" izz="0.0040129019173"/>
-			<origin rpy="0 0 0" xyz="500.224891826 0.00192302092756 -0.000467285335568"/>
+			<origin rpy="0 0 0" xyz="0.224891826 0.00192302092756 -0.000467285335568"/>
 		</inertial>
 		<collision>
@@ -119,5 +119,5 @@
 				<mesh filename="package://abb_common/meshes/irb_120/collision/link_4.stl" scale="0.0254 0.0254 0.0254"/>
 			</geometry>
-			<origin rpy="0 0 0" xyz="500.302187012 0.00151561224702 -0.000313229561613"/>
+			<origin rpy="0 0 0" xyz="0.302187012 0.00151561224702 -0.000313229561613"/>
 		</collision>
 	</link>
@@ -196,5 +196,5 @@
 		<limit effort="300" lower="-2.79" upper="2.79" velocity="5.58"/>
 		<axis xyz="1 0 0"/>
-		<origin rpy="0 0 0" xyz="-500.000188071 0.0701403024607 0.060593734446"/>
+		<origin rpy="0 0 0" xyz="-0.000188071 0.0701403024607 0.060593734446"/>
 	</joint>
 	<joint name="joint5" type="revolute">
@@ -203,5 +203,5 @@
 		<limit effort="300" lower="-2.09" upper="2.09" velocity="5.58"/>
 		<axis xyz="0 0 -1"/>
-		<origin rpy="0 0 0" xyz="500.302186066 0.00151566707848 0.0616850168905"/>
+		<origin rpy="0 0 0" xyz="0.302186066 0.00151566707848 0.0616850168905"/>
 	</joint>
 	<joint name="joint6" type="revolute">

Commit message: Unknown STL scale and coordinate systems.

File: abb/abb_common/urdf/irb_120_macro.xacro (robot description, xacro)
@@ -19,10 +19,4 @@
 			<origin rpy="0 0 0" xyz="0 0 0"/>
 		</inertial>
-		<collision>
-			<geometry>
-				<mesh filename="package://abb_common/meshes/irb_120/collision/base_link.stl" scale="0.0254 0.0254 0.0254"/>
-			</geometry>
-			<origin rpy="0 0 0" xyz="0.04203954 -0.07963916 8.0162399451e-05"/>
-		</collision>
 	</link>
 	<link name="${prefix}link_1">
@@ -43,10 +37,4 @@
 			<origin rpy="0 0 0" xyz="9.92932610521e-05 0.0619125 0.000120146707416"/>
 		</inertial>
-		<collision>
-			<geometry>
-				<mesh filename="package://abb_common/meshes/irb_120/collision/link_1.stl" scale="0.0254 0.0254 0.0254"/>
-			</geometry>
-			<origin rpy="0 0 0" xyz="0 -0.17649952 0"/>
-		</collision>
 	</link>
 	<link name="${prefix}link_2">
@@ -67,10 +55,4 @@
             <origin rpy="0 0 0" xyz="0.000778420420581 0.101238818962 0.0596167646499"/>
 		</inertial>
-		<collision>
-			<geometry>
-				<mesh filename="package://abb_common/meshes/irb_120/collision/link_2.stl" scale="0.0254 0.0254 0.0254"/>
-			</geometry>
-			<origin rpy="0 0 0" xyz="1.54358428872e-06 0.269999754796 0.115499748015"/>
-		</collision>
 	</link>
 	<link name="${prefix}link_3">
@@ -91,10 +73,4 @@
             <origin rpy="0 0 0" xyz="0.0228077138503 0.0579088629114 0.0579265785584"/>
 		</inertial>
-		<collision>
-			<geometry>
-				<mesh filename="package://abb_common/meshes/irb_120/collision/link_3.stl" scale="0.0254 0.0254 0.0254"/>
-			</geometry>
-            <origin rpy="0 0 0" xyz="0.071952848745 -0.0661526901756 0.0589997805382"/>
-		</collision>
 	</link>
 	<link name="${prefix}link_4">
@@ -115,10 +91,4 @@
 			<origin rpy="0 0 0" xyz="0.224891826 0.00192302092756 -0.000467285335568"/>
 		</inertial>
-		<collision>
-			<geometry>
-				<mesh filename="package://abb_common/meshes/irb_120/collision/link_4.stl" scale="0.0254 0.0254 0.0254"/>
-			</geometry>
-			<origin rpy="0 0 0" xyz="0.302187012 0.00151561224702 -0.000313229561613"/>
-		</collision>
 	</link>
 	<link name="${prefix}link_5">
@@ -139,10 +109,4 @@
 			<origin rpy="0 0 0" xyz="-0.00109373496991 6.05486054406e-05 -0.0620361403843"/>
 		</inertial>
-		<collision>
-			<geometry>
-				<mesh filename="package://abb_common/meshes/irb_120/collision/link_5.stl" scale="0.0254 0.0254 0.0254"/>
-			</geometry>
-			<origin rpy="0 0 0" xyz="-0.301998488439 -0.629998750685 -0.0619993114233"/>
-		</collision>
 	</link>
 	<link name="${prefix}link_6">
@@ -163,10 +127,4 @@
 			<origin rpy="0 0 0" xyz="-4.42649390919e-07 0.000169444143624 -0.0070610831163"/>
 		</inertial>
-		<collision>
-			<geometry>
-				<mesh filename="package://abb_common/meshes/irb_120/collision/link_6.stl" scale="0.0254 0.0254 0.0254"/>
-			</geometry>
-			<origin rpy="0 0 0" xyz="-2.74896335695e-07 -8.57788299224e-07 -0.0130000906507"/>
-		</collision>
 	</link>
 	<joint name="joint1" type="revolute">
@@ -174,6 +132,6 @@
 		<child link="${prefix}link_1"/>
 		<limit effort="300" lower="-2.88" upper="2.88" velocity="4.36"/>
-		<axis xyz="0 1 0"/>
-		<origin rpy="-3.14159265359 3.14159265359 3.14159265359" xyz="0.04203954 0.09686036 0"/>
+		<axis xyz="0 0 1"/>
+		<origin rpy="0 0 0" xyz="0 0 0"/>
 	</joint>
 	<joint name="joint2" type="revolute">
@@ -181,6 +139,6 @@
 		<child link="${prefix}link_2"/>
 		<limit effort="300" lower="-1.92" upper="1.92" velocity="4.36"/>
-		<axis xyz="0 0 1"/>
-        <origin rpy="3.14159265359 0 3.14159265359" xyz="0 0.1134999 0.0574996276953"/>
+		<axis xyz="0 1 0"/>
+    <origin rpy="0 0 0" xyz="0 0 0.290"/>
 	</joint>
 	<joint name="joint3" type="revolute">
@@ -188,6 +146,6 @@
 		<child link="${prefix}link_3"/>
 		<limit effort="300" lower="-1.575" upper="1.23" velocity="4.36"/>
-		<axis xyz="0 0 -1"/>
-		<origin rpy="3.14159265359 0 3.14159265359" xyz="0 0.270000153642 0.108"/>
+		<axis xyz="0 1 0"/>
+		<origin rpy="0 0 0" xyz="0 0 0.270"/>
 	</joint>
 	<joint name="joint4" type="revolute">
@@ -196,5 +154,5 @@
 		<limit effort="300" lower="-2.80" upper="2.80" velocity="5.58"/>
 		<axis xyz="1 0 0"/>
-		<origin rpy="0 0 0" xyz="-0.000188071 0.0701403024607 0.060593734446"/>
+		<origin rpy="0 0 0" xyz="0 0 0.70"/>
 	</joint>
 	<joint name="joint5" type="revolute">
@@ -202,6 +160,6 @@
 		<child link="${prefix}link_5"/>
 		<limit effort="300" lower="-2.10" upper="2.10" velocity="5.58"/>
-		<axis xyz="0 0 -1"/>
-		<origin rpy="0 0 0" xyz="0.302186066 0.00151566707848 0.0616850168905"/>
+		<axis xyz="0 -1 0"/>
+		<origin rpy="0 0 0" xyz="0.302 0 0"/>
 	</joint>
 	<joint name="joint6" type="revolute">
@@ -210,5 +168,5 @@
 		<limit effort="300" lower="-6.985" upper="6.985" velocity="7.33"/>
 		<axis xyz="0 0 1"/>
-		<origin rpy="-1.5707961734 0 -1.57079621992" xyz="0.072000865279 0 -0.0620001796247"/>
+		<origin rpy="1.57079632679 0 0" xyz="0.072 0 0"/>
 	</joint>
   </xacro:macro>

Commit message: Simplified joints in irb 120.
Joint specs now properly match dimensioned drawing in IRB-120
datasheet.
Meshes may be slightly misaligned, but joints are all now
guaranteed correct because the assorted strange canceling
offsets are removed and the only transforms are those
specified by the datasheet.
This will require regeneration of the arm nav package(s).

File: abb/abb_common/urdf/irb_120_macro.xacro (robot description, xacro)
@@ -7,5 +7,5 @@
 				<mesh filename="package://abb_common/meshes/irb_120/visual/base_link.stl" scale="0.0254 0.0254 0.0254"/>
 			</geometry>
-			<origin rpy="0 0 0" xyz="0.04203954 -0.07963916 8.0162399451e-05"/>
+			<origin rpy="0 0 0" xyz="0 0 0"/>
       			<material
         			name="abb_orange">
@@ -14,14 +14,9 @@
       			</material>
 		</visual>
-		<inertial>
-			<mass value="6.21503193527"/>
-			<inertia ixx="0.0247271241712" ixy="-0.00130888043627" ixz="-8.0795905152e-05" iyy="0.04723746454" iyz="-8.0325637493e-06" izz="0.049128484834"/>
-			<origin rpy="0 0 0" xyz="0 0 0"/>
-		</inertial>
 		<collision>
 			<geometry>
 				<mesh filename="package://abb_common/meshes/irb_120/collision/base_link.stl" scale="0.0254 0.0254 0.0254"/>
 			</geometry>
-			<origin rpy="0 0 0" xyz="0.04203954 -0.07963916 8.0162399451e-05"/>
+			<origin rpy="0 0 0" xyz="0 0 0"/>
 		</collision>
 	</link>
@@ -31,5 +26,5 @@
 				<mesh filename="package://abb_common/meshes/irb_120/visual/link_1.stl" scale="0.0254 0.0254 0.0254"/>
 			</geometry>
-			<origin rpy="0 0 0" xyz="0 -0.17649952 0"/>
+			<origin rpy="0 0 0" xyz="0 0 0"/>
       			<material
         			name="abb_orange">
@@ -38,14 +33,9 @@
       			</material>
 		</visual>
-		<inertial>
-			<mass value="3.06736850696"/>
-			<inertia ixx="0.0142194659396" ixy="2.31078173317e-05" ixz="-1.08613978372e-05" iyy="0.0104561541196" iyz="1.93410231314e-05" izz="0.0144054074894"/>
-			<origin rpy="0 0 0" xyz="9.92932610521e-05 0.0619125 0.000120146707416"/>
-		</inertial>
 		<collision>
 			<geometry>
 				<mesh filename="package://abb_common/meshes/irb_120/collision/link_1.stl" scale="0.0254 0.0254 0.0254"/>
 			</geometry>
-			<origin rpy="0 0 0" xyz="0 -0.17649952 0"/>
+			<origin rpy="0 0 0" xyz="0 0 0"/>
 		</collision>
 	</link>
@@ -55,5 +45,5 @@
 				<mesh filename="package://abb_common/meshes/irb_120/visual/link_2.stl" scale="0.0254 0.0254 0.0254"/>
 			</geometry>
-            <origin rpy="0 0 0" xyz="1.54358428872e-06 0.269999754796 0.115499748015"/>
+            <origin rpy="0 0 0" xyz="0 0.269999754796 0.0574996276953"/>
       			<material
         			name="abb_orange">
@@ -62,14 +52,9 @@
       			</material>
 		</visual>
-		<inertial>
-			<mass value="3.90875060185"/>
-			<inertia ixx="0.060313948885" ixy="-5.7255892235e-05" ixz="9.0138634014e-06" iyy="0.0259554972424" iyz="-0.00050500074453" izz="0.041571134309"/>
-            <origin rpy="0 0 0" xyz="0.000778420420581 0.101238818962 0.0596167646499"/>
-		</inertial>
 		<collision>
 			<geometry>
 				<mesh filename="package://abb_common/meshes/irb_120/collision/link_2.stl" scale="0.0254 0.0254 0.0254"/>
 			</geometry>
-			<origin rpy="0 0 0" xyz="1.54358428872e-06 0.269999754796 0.115499748015"/>
+			<origin rpy="0 0 0" xyz="0 0.269999754796 0.0574996276953"/>
 		</collision>
 	</link>
@@ -79,5 +64,5 @@
 				<mesh filename="package://abb_common/meshes/irb_120/visual/link_3.stl" scale="0.0254 0.0254 0.0254"/>
 			</geometry>
-            <origin rpy="0 0 0" xyz="0.071952848745 -0.0661526901756 0.0589997805382"/>
+            <origin rpy="0 0 0" xyz="0.071952848745 -0.0661526901756 0"/>
       			<material
         			name="abb_orange">
@@ -86,14 +71,9 @@
       			</material>
 		</visual>
-		<inertial>
-			<mass value="2.94383262499"/>
-			<inertia ixx="0.0083145487625" ixy="-0.00142864798126" ixz="-7.9926773262e-05" iyy="0.0126560235034" iyz="-0.000181719383164" izz="0.016713669618"/>
-            <origin rpy="0 0 0" xyz="0.0228077138503 0.0579088629114 0.0579265785584"/>
-		</inertial>
 		<collision>
 			<geometry>
 				<mesh filename="package://abb_common/meshes/irb_120/collision/link_3.stl" scale="0.0254 0.0254 0.0254"/>
 			</geometry>
-            <origin rpy="0 0 0" xyz="0.071952848745 -0.0661526901756 0.0589997805382"/>
+            <origin rpy="0 0 0" xyz="0.071952848745 -0.0661526901756 0"/>
 		</collision>
 	</link>
@@ -110,14 +90,9 @@
       			</material>
 		</visual>
-		<inertial>
-			<mass value="1.32790527095"/>
-			<inertia ixx="0.00284579825479" ixy="1.64819596414e-05" ixz="-2.12443634431e-05" iyy="0.0052535657425" iyz="1.31403377384e-05" izz="0.0040129019173"/>
-			<origin rpy="0 0 0" xyz="0.224891826 0.00192302092756 -0.000467285335568"/>
-		</inertial>
 		<collision>
 			<geometry>
 				<mesh filename="package://abb_common/meshes/irb_120/collision/link_4.stl" scale="0.0254 0.0254 0.0254"/>
 			</geometry>
-			<origin rpy="0 0 0" xyz="0.302187012 0.00151561224702 -0.000313229561613"/>
+			<origin rpy="0 0 0" xyz="0.302187012 0.00151561224702 0"/>
 		</collision>
 	</link>
@@ -127,5 +102,5 @@
 				<mesh filename="package://abb_common/meshes/irb_120/visual/link_5.stl" scale="0.0254 0.0254 0.0254"/>
 			</geometry>
-			<origin rpy="0 0 0" xyz="-0.301998488439 -0.629998750685 -0.0619993114233"/>
+			<origin rpy="0 0 0" xyz="-0.301998488439 -0.629998750685 0"/>
       			<material
         			name="abb_orange">
@@ -134,14 +109,9 @@
       			</material>
 		</visual>
-		<inertial>
-			<mass value="0.546633236934"/>
-			<inertia ixx="0.00040430142646" ixy="-8.1520474364e-07" ixz="1.6167316339e-06" iyy="0.00081538617858" iyz="-1.38898103591e-08" izz="0.00089215071642"/>
-			<origin rpy="0 0 0" xyz="-0.00109373496991 6.05486054406e-05 -0.0620361403843"/>
-		</inertial>
 		<collision>
 			<geometry>
 				<mesh filename="package://abb_common/meshes/irb_120/collision/link_5.stl" scale="0.0254 0.0254 0.0254"/>
 			</geometry>
-			<origin rpy="0 0 0" xyz="-0.301998488439 -0.629998750685 -0.0619993114233"/>
+			<origin rpy="0 0 0" xyz="-0.301998488439 -0.629998750685 0"/>
 		</collision>
 	</link>
@@ -151,21 +121,16 @@
 				<mesh filename="package://abb_common/meshes/irb_120/visual/link_6.stl" scale="0.0254 0.0254 0.0254"/>
 			</geometry>
-			<origin rpy="0 0 0" xyz="-2.74896335695e-07 -8.57788299224e-07 -0.0130000906507"/>
+			<origin rpy="0 0 0" xyz="0 0 -0.0130000906507"/>
       			<material
-        			name="abb_orange">
+        			name="abb_black">
         			<color
-          			rgba="1 0.43 0 1" />
+          			rgba="0 0 0 1" />
       			</material>
 		</visual>
-		<inertial>
-			<mass value="0.0136784407912"/>
-			<inertia ixx="1.65768910842e-06" ixy="-3.0670406059e-12" ixz="8.9225606574e-11" iyy="1.69424824883e-06" iyz="-7.6624364717e-09" izz="2.9767913551e-06"/>
-			<origin rpy="0 0 0" xyz="-4.42649390919e-07 0.000169444143624 -0.0070610831163"/>
-		</inertial>
 		<collision>
 			<geometry>
 				<mesh filename="package://abb_common/meshes/irb_120/collision/link_6.stl" scale="0.0254 0.0254 0.0254"/>
 			</geometry>
-			<origin rpy="0 0 0" xyz="-2.74896335695e-07 -8.57788299224e-07 -0.0130000906507"/>
+			<origin rpy="0 0 0" xyz="0 0 -0.0130000906507"/>
 		</collision>
 	</link>
@@ -175,5 +140,5 @@
 		<limit effort="300" lower="-2.88" upper="2.88" velocity="4.36"/>
 		<axis xyz="0 1 0"/>
-		<origin rpy="-3.14159265359 3.14159265359 3.14159265359" xyz="0.04203954 0.09686036 0"/>
+		<origin rpy="-3.14159265359 3.14159265359 3.14159265359" xyz="0 0 0"/>
 	</joint>
 	<joint name="joint2" type="revolute">
@@ -182,5 +147,5 @@
 		<limit effort="300" lower="-1.92" upper="1.92" velocity="4.36"/>
 		<axis xyz="0 0 1"/>
-        <origin rpy="3.14159265359 0 3.14159265359" xyz="0 0.1134999 0.0574996276953"/>
+        <origin rpy="3.14159265359 0 3.14159265359" xyz="0 0.290 0"/>
 	</joint>
 	<joint name="joint3" type="revolute">
@@ -189,5 +154,5 @@
 		<limit effort="300" lower="-1.575" upper="1.23" velocity="4.36"/>
 		<axis xyz="0 0 -1"/>
-		<origin rpy="3.14159265359 0 3.14159265359" xyz="0 0.270000153642 0.108"/>
+		<origin rpy="3.14159265359 0 3.14159265359" xyz="0 0.270 0"/>
 	</joint>
 	<joint name="joint4" type="revolute">
@@ -196,5 +161,5 @@
 		<limit effort="300" lower="-2.80" upper="2.80" velocity="5.58"/>
 		<axis xyz="1 0 0"/>
-		<origin rpy="0 0 0" xyz="-0.000188071 0.0701403024607 0.060593734446"/>
+		<origin rpy="0 0 0" xyz="0 0.070 0"/>
 	</joint>
 	<joint name="joint5" type="revolute">
@@ -203,5 +168,5 @@
 		<limit effort="300" lower="-2.10" upper="2.10" velocity="5.58"/>
 		<axis xyz="0 0 -1"/>
-		<origin rpy="0 0 0" xyz="0.302186066 0.00151566707848 0.0616850168905"/>
+		<origin rpy="0 0 0" xyz="0.302 0 0"/>
 	</joint>
 	<joint name="joint6" type="revolute">
@@ -210,5 +175,5 @@
 		<limit effort="300" lower="-6.985" upper="6.985" velocity="7.33"/>
 		<axis xyz="0 0 1"/>
-		<origin rpy="-1.5707961734 0 -1.57079621992" xyz="0.072000865279 0 -0.0620001796247"/>
+		<origin rpy="-1.5707961734 0 -1.57079621992" xyz="0.072 0 0"/>
 	</joint>
   </xacro:macro>

Commit message: Flipped link2 over.

File: abb/abb_common/urdf/irb_120_macro.xacro (robot description, xacro)
@@ -45,5 +45,5 @@
 				<mesh filename="package://abb_common/meshes/irb_120/visual/link_2.stl" scale="0.0254 0.0254 0.0254"/>
 			</geometry>
-            <origin rpy="0 0 0" xyz="0 0.269999754796 0.0574996276953"/>
+            <origin rpy="0 3.14159 0" xyz="0 0.269999754796 -0.0574996276953"/>
       			<material
         			name="abb_orange">
@@ -56,5 +56,5 @@
 				<mesh filename="package://abb_common/meshes/irb_120/collision/link_2.stl" scale="0.0254 0.0254 0.0254"/>
 			</geometry>
-			<origin rpy="0 0 0" xyz="0 0.269999754796 0.0574996276953"/>
+			<origin rpy="0 3.14159 0" xyz="0 0.269999754796 -0.0574996276953"/>
 		</collision>
 	</link>
