Commit message: Trying to figure out the ik solver.
Wheeeeeee

File: abb/abb_common/urdf/irb_120.urdf (robot description, URDF)
Before this commit: robot irb_120, 7 links, 6 joints
Links:
- link base_link: mass 6.21503193527 -> None
- link link_1: mass 3.06736850696 -> None
- link link_2: mass 3.90875060185 -> None
- link link_3: mass 2.94383262499 -> None
- link link_4: mass 1.32790527095 -> None
- link link_5: mass 0.546633236934 -> None
- link link_6: mass 0.0136784407912 -> None
Joints:
- joint joint1: origin xyz=0.04203954 0.09686036 0 rpy=-3.14159265359 3.14159265359 3.14159265359 -> xyz=0 0 0 rpy=-3.14159265359 3.14159265359 3.14159265359
- joint joint2: origin xyz=0 0.1134999 0.0574996276953 rpy=3.14159265359 0 3.14159265359 -> xyz=0 0.290 0 rpy=3.14159265359 0 3.14159265359
- joint joint3: limit lower=-1.92 upper=1.22 effort=300 velocity=4.36 -> lower=-1.575 upper=1.23 effort=300 velocity=4.36; origin xyz=0 0.270000153642 0.108 rpy=3.14159265359 0 3.14159265359 -> xyz=0 0.270 0 rpy=3.14159265359 0 3.14159265359
- joint joint4: limit lower=-2.79 upper=2.79 effort=300 velocity=5.58 -> lower=-2.80 upper=2.80 effort=300 velocity=5.58; origin xyz=-500.000188071 0.0701403024607 0.060593734446 rpy=0 0 0 -> xyz=0 0.070 0 rpy=0 0 0
- joint joint5: limit lower=-2.09 upper=2.09 effort=300 velocity=5.58 -> lower=-2.10 upper=2.10 effort=300 velocity=5.58; origin xyz=500.302186066 0.00151566707848 0.0616850168905 rpy=0 0 0 -> xyz=0.302 0.001 0 rpy=0 0 0
- joint joint6: limit lower=-6.98 upper=6.98 effort=300 velocity=7.33 -> lower=-6.985 upper=6.985 effort=300 velocity=7.33; origin xyz=0.072000865279 0 -0.0620001796247 rpy=-1.5707961734 0 -1.57079621992 -> xyz=0.072 0 0 rpy=-1.5707961734 0 -1.57079621992

File: abb/abb_common/urdf/irb_120_macro.xacro (robot description, xacro)
@@ -168,5 +168,5 @@
 		<limit effort="300" lower="-2.10" upper="2.10" velocity="5.58"/>
 		<axis xyz="0 0 -1"/>
-		<origin rpy="0 0 0" xyz="0.302 0 0"/>
+		<origin rpy="0 0 0" xyz="0.302 0.001 0"/>
 	</joint>
 	<joint name="joint6" type="revolute">
