Commit message: added arm navigation packages for both arms
git-svn-id: http://swri-ros-pkg.googlecode.com/svn/trunk@688 076cdf4d-ed99-c8c1-5d01-9bc0d27e81bd

File: fanuc/fanuc_config/urdf/M16iB20_macro.xacro (robot description, xacro)
@@ -317,5 +317,5 @@
 		    <limit
 		      lower="-1.5708"
-		      upper="2.7925"
+		      upper="1.9"
 		      effort="0"
 		      velocity="0" />
@@ -343,6 +343,6 @@
 		      xyz="0 1 0" />
 		    <limit
-		      lower="-2.9671"
-		      upper="5.0615"
+		      lower="-4.21"
+		      upper="1.45"
 		      effort="0"
 		      velocity="0" />

File: fanuc/fanuc_config/urdf/m_430iA2F_macro.xacro (robot description, xacro)
@@ -109,6 +109,6 @@
         <joint name="${prefix}joint_1" type="revolute">
             <origin xyz="-6.0758E-19 1.2493E-16 0.44" rpy="0 0 0" />
-            <parent link="base_link" />
-            <child link="link_1" />
+            <parent link="${prefix}base_link" />
+            <child link="${prefix}link_1" />
             <axis xyz="0 0 1" />
             <limit lower="-3.1415" upper="3.1415" effort="0"
@@ -121,6 +121,6 @@
         <joint name="${prefix}joint_2" type="revolute">
             <origin xyz="-1.4097E-17 0.171 -4.4409E-16" rpy="0 0 0" />
-            <parent link="link_1" />
-            <child link="link_2" />
+            <parent link="${prefix}link_1" />
+            <child link="${prefix}link_2" />
             <axis xyz="0 1 0" />
             <limit lower="-2.00707" upper="2.00707" effort="0"
@@ -134,6 +134,6 @@
             <!-- origin xyz="1.2197E-19 -0.171 0.403" rpy="0 0 0" / -->
             <origin xyz="1.2197E-19 -0.171 0.350" rpy="0 0 0" />
-            <parent link="link_2" />
-            <child link="link_3" />
+            <parent link="${prefix}link_2" />
+            <child link="${prefix}link_3" />
             <axis xyz="0 1 0" />
             <limit lower="-1.771457" upper="1.771457" effort="0"
@@ -147,6 +147,6 @@
             <!-- origin xyz="-2.6075E-17 -0.06 0.497" rpy="0 0 0" / -->
             <origin xyz="-2.6075E-17 -0.06 0.55" rpy="0 0 0" />
-            <parent link="link_3" />
-            <child link="link_4" />
+            <parent link="${prefix}link_3" />
+            <child link="${prefix}link_4" />
             <axis xyz="0 1 0" />
             <limit lower="-2.617917" upper="2.617917" effort="0"
@@ -159,6 +159,6 @@
 		<joint name="${prefix}joint_5" type="revolute">
 			<origin xyz="1.4734E-16 -0.035 0.065" rpy="0 0 0" />
-			<parent link="link_4" />
-			<child link="link_5" />
+			<parent link="${prefix}link_4" />
+			<child link="${prefix}link_5" />
 			<axis xyz="0 0 1" />
 			<limit lower="-4.71225" upper="4.71225" effort="0"

File: motoman/motoman_config/cfg/sia20d_mesh_macro.xacro (robot description, xacro)
@@ -1,2 +1,3 @@
+<?xml version="1.0" ?>
 <robot xmlns:xacro="http://ros.org/wiki/xacro">
 	<xacro:macro name="sia20d_mesh" params="prefix">
@@ -135,6 +136,6 @@
 		<!-- joint list -->
 		<joint name="${prefix}joint_s" type="revolute">
-			<parent link="base_link"/>
-			<child link="link_s"/>
+			<parent link="${prefix}base_link"/>
+			<child link="${prefix}link_s"/>
 			<origin xyz="0 0 0.41" rpy="0 0 0"/>
 			<axis xyz="0 0 1" />
@@ -142,6 +143,6 @@
 		</joint>
 		<joint name="${prefix}joint_l" type="revolute">
-			<parent link="link_s"/>
-			<child link="link_l"/>
+			<parent link="${prefix}link_s"/>
+			<child link="${prefix}link_l"/>
 			<origin xyz="0 0 0" rpy="0 0 0"/>
 			<axis xyz="0 1 0" />
@@ -149,6 +150,6 @@
 		</joint>
 		<joint name="${prefix}joint_e" type="revolute">
-			<parent link="link_l"/>
-			<child link="link_e"/>
+			<parent link="${prefix}link_l"/>
+			<child link="${prefix}link_e"/>
 			<origin xyz="0 0 0.49" rpy="0 0 0"/>
 			<axis xyz="0 0 1" />
@@ -156,6 +157,6 @@
 		</joint>
 		<joint name="${prefix}joint_u" type="revolute">
-			<parent link="link_e"/>
-			<child link="link_u"/>
+			<parent link="${prefix}link_e"/>
+			<child link="${prefix}link_u"/>
 			<origin xyz="0 0 0" rpy="0 0 0"/>
 			<axis xyz="0 -1 0" />
@@ -163,6 +164,6 @@
 		</joint>
 		<joint name="${prefix}joint_r" type="revolute">
-			<parent link="link_u"/>
-			<child link="link_r"/>
+			<parent link="${prefix}link_u"/>
+			<child link="${prefix}link_r"/>
 			<origin xyz="0 0 0.420" rpy="0 0 0"/>
 			<axis xyz="0 0 -1" />
@@ -170,6 +171,6 @@
 		</joint>
 		<joint name="${prefix}joint_b" type="revolute">
-			<parent link="link_r"/>
-			<child link="link_b"/>
+			<parent link="${prefix}link_r"/>
+			<child link="${prefix}link_b"/>
 			<origin xyz="0 0 0" rpy="0 0 0"/>
 			<axis xyz="0 -1 0" />
@@ -177,6 +178,6 @@
 		</joint>
 		<joint name="${prefix}joint_t" type="revolute">
-			<parent link="link_b"/>
-			<child link="link_t"/>
+			<parent link="${prefix}link_b"/>
+			<child link="${prefix}link_t"/>
 			<origin xyz="0 0 0.18" rpy="0 0 0"/>
 			<axis xyz="0 0 -1" />
