Commit message: Added vacuum gripper model .stl's to replace the box which was representing the gripper
git-svn-id: http://swri-ros-pkg.googlecode.com/svn/trunk@712 076cdf4d-ed99-c8c1-5d01-9bc0d27e81bd

File: mantis/mantis_config/urdf/mantis.urdf (robot description, URDF)
Before this commit: robot motoman_vacumm, 21 links, 20 joints
Links:
- link palm: geometry collision mesh filename=package://mantis_config/config/meshes/vacuum_gripper.stl; visual mesh filename=package://mantis_config/config/meshes/vacuum_gripper.STL

File: mantis/mantis_config/urdf/vacuum_gripper_block.xacro (robot description, xacro)
@@ -4,16 +4,16 @@
 		<link name="${prefix}palm">
 			<visual>
-				<origin xyz="0 0.036 -0.1" rpy="0 0 0"/>
+				<origin xyz="0 0.036 -0.0473" rpy="0 0 0"/>
 				<geometry>
-					<mesh filename="package://mantis_config/config/meshes/vacuum_gripper.STL" />
+					<box size="0.044 0.088 0.0946"/>
 				</geometry>
-				<material name="silver">
-					<color rgba="0.8 0.8 0.8 1"/>
+				<material name="another_blue1">
+					<color rgba="0.40 0.40 0.80 1"/>
 				</material>
 			</visual>
 			<collision>
-				<origin xyz="0 0.036 -0.1" rpy="0 0 0"/>
+				<origin xyz="0 0.036 -0.0473" rpy="0 0 0"/>
 				<geometry>
-					<mesh filename="package://mantis_config/config/meshes/vacuum_gripper.stl" />
+					<box size="0.044 0.088 0.0946"/>
 				</geometry>
 				<material name="another_blue2">
