Commit message: launch files for sia20d navigation updated
git-svn-id: http://swri-ros-pkg.googlecode.com/svn/trunk@726 076cdf4d-ed99-c8c1-5d01-9bc0d27e81bd

File: mantis/mantis_config/urdf/mantis_dual_arm_workspace.urdf (robot description, URDF)
Before this commit: robot mantis_dual, 49 links, 48 joints
Links:
- removed link sia20d_arm/base_link
- removed link sia20d_arm/coupler
- removed link sia20d_arm/kinect
- removed link sia20d_arm/kinect_frame
- removed link sia20d_arm/kinect_ir_link
- removed link sia20d_arm/kinect_ir_optical_frame
- removed link sia20d_arm/kinect_keepout
- removed link sia20d_arm/kinect_rgb_link
- removed link sia20d_arm/kinect_rgb_optical_frame
- removed link sia20d_arm/link_b
- removed link sia20d_arm/link_e
- removed link sia20d_arm/link_l
- removed link sia20d_arm/link_r
- removed link sia20d_arm/link_s
- removed link sia20d_arm/link_t
- removed link sia20d_arm/link_u
- removed link sia20d_arm/palm
- removed link ur5_arm/base_link
- removed link ur5_arm/ee_link
- removed link ur5_arm/forearm_link
- removed link ur5_arm/gripper_body
- removed link ur5_arm/gripper_frame
- removed link ur5_arm/kinect
- removed link ur5_arm/kinect_frame
- removed link ur5_arm/kinect_ir_link
- removed link ur5_arm/kinect_ir_optical_frame
- removed link ur5_arm/kinect_keepout
- removed link ur5_arm/kinect_rgb_link
- removed link ur5_arm/kinect_rgb_optical_frame
- removed link ur5_arm/shoulder_link
- removed link ur5_arm/tcp_frame
- removed link ur5_arm/upper_arm_link
- removed link ur5_arm/wrist_1_link
- removed link ur5_arm/wrist_2_link
- removed link ur5_arm/wrist_3_link
- added link sia20d_arm_base_link; collision mesh filename=package://motoman_config/meshes/sia20d/collision/MOTOMAN_BA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; visual mesh filename=package://motoman_config/meshes/sia20d/visual/MOTOMAN_BASE.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
- added link sia20d_arm_coupler; collision mesh filename=package://longhorn/meshes/coupler/collision/COUPLER.stl; visual mesh filename=package://longhorn/meshes/coupler/visual/COUPLER.stl
- added link sia20d_arm_kinect; collision box size=0.36 0.28 0.22
- added link sia20d_arm_kinect_frame; collision box size=0.064 0.28 0.04; visual box size=0.064 0.28 0.04
- added link sia20d_arm_kinect_ir_link; visual sphere radius=0.0005
- added link sia20d_arm_kinect_ir_optical_frame
- added link sia20d_arm_kinect_keepout; collision box size=0.2 0.32 0.48
- added link sia20d_arm_kinect_rgb_link; visual sphere radius=0.0005
- added link sia20d_arm_kinect_rgb_optical_frame
- added link sia20d_arm_link_b; collision mesh filename=package://motoman_config/meshes/sia20d/collision/MOTOMAN_AX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; visual mesh filename=package://motoman_config/meshes/sia20d/visual/MOTOMAN_AXIS_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
- added link sia20d_arm_link_e; collision mesh filename=package://motoman_config/meshes/sia20d/collision/MOTOMAN_AX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; visual mesh filename=package://motoman_config/meshes/sia20d/visual/MOTOMAN_AXIS_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
- added link sia20d_arm_link_l; collision mesh filename=package://motoman_config/meshes/sia20d/collision/MOTOMAN_AX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; visual mesh filename=package://motoman_config/meshes/sia20d/visual/MOTOMAN_AXIS_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
- added link sia20d_arm_link_r; collision mesh filename=package://motoman_config/meshes/sia20d/collision/MOTOMAN_AX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; visual mesh filename=package://motoman_config/meshes/sia20d/visual/MOTOMAN_AXIS_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
- added link sia20d_arm_link_s; collision mesh filename=package://motoman_config/meshes/sia20d/collision/MOTOMAN_AX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; visual mesh filename=package://motoman_config/meshes/sia20d/visual/MOTOMAN_AXIS_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
- added link sia20d_arm_link_t; collision mesh filename=package://motoman_config/meshes/sia20d/collision/MOTOMAN_AX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; visual mesh filename=package://motoman_config/meshes/sia20d/visual/MOTOMAN_AXIS_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
- added link sia20d_arm_link_u; collision mesh filename=package://motoman_config/meshes/sia20d/collision/MOTOMAN_AX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; visual mesh filename=package://motoman_config/meshes/sia20d/visual/MOTOMAN_AXIS_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
- added link sia20d_arm_palm; collision box size=0.044 0.088 0.0946; visual box size=0.044 0.088 0.0946
- added link ur5_arm_base_link, mass 4.0; visual mesh filename=package://ur5_description/meshes/Base.dae
- added link ur5_arm_ee_link
- added link ur5_arm_forearm_link, mass 2.275; collision cylinder length=0.39225 radius=0.04; visual mesh filename=package://ur5_description/meshes/Forearm.dae
- added link ur5_arm_gripper_body; collision box size=0.044 0.088 0.0946; visual box size=0.044 0.088 0.0946
- added link ur5_arm_gripper_frame
- added link ur5_arm_kinect; collision box size=0.36 0.28 0.22
- added link ur5_arm_kinect_frame; collision box size=0.064 0.28 0.04; visual box size=0.064 0.28 0.04
- added link ur5_arm_kinect_ir_link; visual sphere radius=0.0005
- added link ur5_arm_kinect_ir_optical_frame
- added link ur5_arm_kinect_keepout; collision box size=0.2 0.32 0.48
- added link ur5_arm_kinect_rgb_link; visual sphere radius=0.0005
- added link ur5_arm_kinect_rgb_optical_frame
- added link ur5_arm_shoulder_link, mass 3.7; collision cylinder length=0.16 radius=0.06; visual mesh filename=package://ur5_description/meshes/Shoulder.dae
- added link ur5_arm_tcp_frame
- added link ur5_arm_upper_arm_link, mass 8.393; collision cylinder length=0.425 radius=0.054; visual mesh filename=package://ur5_description/meshes/UpperArm.dae
- added link ur5_arm_wrist_1_link, mass 1.219; collision cylinder length=0.1488 radius=0.045; visual mesh filename=package://ur5_description/meshes/Wrist1.dae
- added link ur5_arm_wrist_2_link, mass 1.219; collision cylinder length=0.15144 radius=0.045; visual mesh filename=package://ur5_description/meshes/Wrist2.dae
- added link ur5_arm_wrist_3_link, mass 0.1879; collision cylinder length=0.135795 radius=0.045; visual mesh filename=package://ur5_description/meshes/Wrist3.dae
Joints:
- removed joint sia20d_arm/joint_b
- removed joint sia20d_arm/joint_e
- removed joint sia20d_arm/joint_l
- removed joint sia20d_arm/joint_r
- removed joint sia20d_arm/joint_s
- removed joint sia20d_arm/joint_t
- removed joint sia20d_arm/joint_u
- removed joint sia20d_arm/kinect_frame_joint
- removed joint sia20d_arm/kinect_ir_joint
- removed joint sia20d_arm/kinect_ir_optical_frame_joint
- removed joint sia20d_arm/kinect_rgb_joint
- removed joint sia20d_arm/kinect_rgb_optical_frame_joint
- removed joint sia20d_arm/workcell_frame_to_kinect
- removed joint sia20d_arm/workcell_frame_to_kinect_keepout
- removed joint ur5_arm/ee_fixed_joint
- removed joint ur5_arm/elbow_joint
- removed joint ur5_arm/gripper_to_palm
- removed joint ur5_arm/gripper_to_tcp
- removed joint ur5_arm/kinect_frame_joint
- removed joint ur5_arm/kinect_ir_joint
- removed joint ur5_arm/kinect_ir_optical_frame_joint
- removed joint ur5_arm/kinect_rgb_joint
- removed joint ur5_arm/kinect_rgb_optical_frame_joint
- removed joint ur5_arm/shoulder_lift_joint
- removed joint ur5_arm/shoulder_pan_joint
- removed joint ur5_arm/workcell_frame_to_kinect
- removed joint ur5_arm/workcell_frame_to_kinect_keepout
- removed joint ur5_arm/wrist_1_joint
- removed joint ur5_arm/wrist_2_joint
- removed joint ur5_arm/wrist_3_joint
- added joint sia20d_arm_joint_b: type revolute, parent sia20d_arm_link_r, child sia20d_arm_link_b, origin xyz=0 0 0 rpy=0 0 0, axis 0 -1 0, limit lower=-1.91 upper=1.91 effort=100 velocity=3.48
- added joint sia20d_arm_joint_e: type revolute, parent sia20d_arm_link_l, child sia20d_arm_link_e, origin xyz=0 0 0.49 rpy=0 0 0, axis 0 0 1, limit lower=-2.96 upper=2.96 effort=100 velocity=2.96
- added joint sia20d_arm_joint_l: type revolute, parent sia20d_arm_link_s, child sia20d_arm_link_l, origin xyz=0 0 0 rpy=0 0 0, axis 0 1 0, limit lower=-1.91 upper=1.91 effort=100 velocity=2.26
- added joint sia20d_arm_joint_r: type revolute, parent sia20d_arm_link_u, child sia20d_arm_link_r, origin xyz=0 0 0.420 rpy=0 0 0, axis 0 0 -1, limit lower=-3.1416 upper=3.1416 effort=100 velocity=3.48
- added joint sia20d_arm_joint_s: type revolute, parent sia20d_arm_base_link, child sia20d_arm_link_s, origin xyz=0 0 0.41 rpy=0 0 0, axis 0 0 1, limit lower=-3.1416 upper=3.1416 effort=100 velocity=2.26
- added joint sia20d_arm_joint_t: type revolute, parent sia20d_arm_link_b, child sia20d_arm_link_t, origin xyz=0 0 0.18 rpy=0 0 0, axis 0 0 -1, limit lower=-3.1416 upper=3.1416 effort=100 velocity=6.97
- added joint sia20d_arm_joint_u: type revolute, parent sia20d_arm_link_e, child sia20d_arm_link_u, origin xyz=0 0 0 rpy=0 0 0, axis 0 -1 0, limit lower=-2.26 upper=2.26 effort=100 velocity=2.96
- added joint sia20d_arm_kinect_frame_joint: type fixed, parent sia20d_arm_kinect, child sia20d_arm_kinect_frame, origin xyz=0 0 0 rpy=0 0 0
- added joint sia20d_arm_kinect_ir_joint: type fixed, parent sia20d_arm_kinect_frame, child sia20d_arm_kinect_ir_link, origin xyz=0 0 0 rpy=0 0 0
- added joint sia20d_arm_kinect_ir_optical_frame_joint: type fixed, parent sia20d_arm_kinect_ir_link, child sia20d_arm_kinect_ir_optical_frame, origin xyz=0 0 0 rpy=-1.57 0 -1.57
- added joint sia20d_arm_kinect_rgb_joint: type fixed, parent sia20d_arm_kinect_ir_link, child sia20d_arm_kinect_rgb_link, origin xyz=0 -0.03 0 rpy=0 0 0
- added joint sia20d_arm_kinect_rgb_optical_frame_joint: type fixed, parent sia20d_arm_kinect_rgb_link, child sia20d_arm_kinect_rgb_optical_frame, origin xyz=0 0 0 rpy=-1.57 0 -1.57
- added joint sia20d_arm_workcell_frame_to_kinect: type fixed, parent workcell_frame, child sia20d_arm_kinect, origin xyz=1.2 0 0.4 rpy=0 0.5235 3.147
- added joint sia20d_arm_workcell_frame_to_kinect_keepout: type fixed, parent workcell_frame, child sia20d_arm_kinect_keepout, origin xyz=1.2 0 0.24 rpy=0 0 3.147
- added joint ur5_arm_ee_fixed_joint: type fixed, parent ur5_arm_wrist_3_link, child ur5_arm_ee_link, origin xyz=0.0 0.0823 0.0 rpy=0.0 0.0 1.570796325
- added joint ur5_arm_elbow_joint: type revolute, parent ur5_arm_upper_arm_link, child ur5_arm_forearm_link, origin xyz=0.0 -0.1197 0.425 rpy=0.0 0.0 0.0, axis 0.0 1.0 0.0, limit lower=-6.2831853 upper=6.2831853 effort=10.0 velocity=3.14159265
- added joint ur5_arm_gripper_to_palm: type fixed, parent ur5_arm_gripper_frame, child ur5_arm_gripper_body, origin xyz=0 0 0.0473 rpy=0 0 0
- added joint ur5_arm_gripper_to_tcp: type fixed, parent ur5_arm_gripper_frame, child ur5_arm_tcp_frame, origin xyz=0.022 0 0.0946 rpy=0 0 0
- added joint ur5_arm_kinect_frame_joint: type fixed, parent ur5_arm_kinect, child ur5_arm_kinect_frame, origin xyz=0 0 0 rpy=0 0 0
- added joint ur5_arm_kinect_ir_joint: type fixed, parent ur5_arm_kinect_frame, child ur5_arm_kinect_ir_link, origin xyz=0 0 0 rpy=0 0 0
- added joint ur5_arm_kinect_ir_optical_frame_joint: type fixed, parent ur5_arm_kinect_ir_link, child ur5_arm_kinect_ir_optical_frame, origin xyz=0 0 0 rpy=-1.57 0 -1.57
- added joint ur5_arm_kinect_rgb_joint: type fixed, parent ur5_arm_kinect_ir_link, child ur5_arm_kinect_rgb_link, origin xyz=0 -0.03 0 rpy=0 0 0
- added joint ur5_arm_kinect_rgb_optical_frame_joint: type fixed, parent ur5_arm_kinect_rgb_link, child ur5_arm_kinect_rgb_optical_frame, origin xyz=0 0 0 rpy=-1.57 0 -1.57
- added joint ur5_arm_shoulder_lift_joint: type revolute, parent ur5_arm_shoulder_link, child ur5_arm_upper_arm_link, origin xyz=0.0 0.13585 0.0 rpy=0.0 1.570796325 0.0, axis 0.0 1.0 0.0, limit lower=-6.2831853 upper=6.2831853 effort=10.0 velocity=3.14159265
- added joint ur5_arm_shoulder_pan_joint: type revolute, parent ur5_arm_base_link, child ur5_arm_shoulder_link, origin xyz=0.0 0.0 0.089159 rpy=0.0 0.0 0.0, axis 0.0 0.0 1.0, limit lower=-6.2831853 upper=6.2831853 effort=10.0 velocity=3.14159265
- added joint ur5_arm_workcell_frame_to_kinect: type fixed, parent workcell_frame, child ur5_arm_kinect, origin xyz=-1.2 0 0.4 rpy=0 0.5235 0
- added joint ur5_arm_workcell_frame_to_kinect_keepout: type fixed, parent workcell_frame, child ur5_arm_kinect_keepout, origin xyz=-1.2 0 0.24 rpy=0 0 0
- added joint ur5_arm_wrist_1_joint: type revolute, parent ur5_arm_forearm_link, child ur5_arm_wrist_1_link, origin xyz=0.0 0.0 0.39225 rpy=0.0 1.570796325 0.0, axis 0.0 1.0 0.0, limit lower=-6.2831853 upper=6.2831853 effort=10.0 velocity=3.14159265
- added joint ur5_arm_wrist_2_joint: type revolute, parent ur5_arm_wrist_1_link, child ur5_arm_wrist_2_link, origin xyz=0.0 0.093 0.0 rpy=0.0 0.0 0.0, axis 0.0 0.0 1.0, limit lower=-6.2831853 upper=6.2831853 effort=10.0 velocity=3.14159265
- added joint ur5_arm_wrist_3_joint: type revolute, parent ur5_arm_wrist_2_link, child ur5_arm_wrist_3_link, origin xyz=0.0 0.0 0.09465 rpy=0.0 0.0 0.0, axis 0.0 1.0 0.0, limit lower=-6.2831853 upper=6.2831853 effort=10.0 velocity=3.14159265
- joint coupler-hand: child sia20d_arm/palm -> sia20d_arm_palm; parent sia20d_arm/coupler -> sia20d_arm_coupler
- joint sia20d_to_workcell: child sia20d_arm/base_link -> sia20d_arm_base_link
- joint tool-coupler: child sia20d_arm/coupler -> sia20d_arm_coupler; parent sia20d_arm/link_t -> sia20d_arm_link_t
- joint ur5_to_gripper: child ur5_arm/gripper_frame -> ur5_arm_gripper_frame; parent ur5_arm/ee_link -> ur5_arm_ee_link
- joint ur5_to_stand: child ur5_arm/base_link -> ur5_arm_base_link

File: mantis/mantis_config/urdf/mantis_dual_arm_workspace.xacro (robot description, xacro)
@@ -11,6 +11,6 @@
 	<xacro:property name="workcell_height" value="1"/>
 	<xacro:property name="vacuum_gripper_width" value="0.088"/>
-	<xacro:property name="arm1_prefix" value="sia20d_arm/"/>
-	<xacro:property name="arm2_prefix" value="ur5_arm/"/>
+	<xacro:property name="arm1_prefix" value="sia20d_arm_"/>
+	<xacro:property name="arm2_prefix" value="ur5_arm_"/>
 	<xacro:property name="arm1_name" value="sia20d"/>
 	<xacro:property name="arm2_name" value="ur5"/>

File: mantis/mantis_config/urdf/mantis_sia20d.urdf (robot description, URDF)
Before this commit: robot mantis_sia20d, 23 links, 22 joints
Links:
- removed link sia20d_arm/base_link
- removed link sia20d_arm/coupler
- removed link sia20d_arm/kinect
- removed link sia20d_arm/kinect_frame
- removed link sia20d_arm/kinect_ir_link
- removed link sia20d_arm/kinect_ir_optical_frame
- removed link sia20d_arm/kinect_keepout
- removed link sia20d_arm/kinect_rgb_link
- removed link sia20d_arm/kinect_rgb_optical_frame
- removed link sia20d_arm/link_b
- removed link sia20d_arm/link_e
- removed link sia20d_arm/link_l
- removed link sia20d_arm/link_r
- removed link sia20d_arm/link_s
- removed link sia20d_arm/link_t
- removed link sia20d_arm/link_u
- removed link sia20d_arm/palm
- added link sia20d_arm_base_link; collision mesh filename=package://motoman_config/meshes/sia20d/collision/MOTOMAN_BA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; visual mesh filename=package://motoman_config/meshes/sia20d/visual/MOTOMAN_BASE.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
- added link sia20d_arm_coupler; collision mesh filename=package://longhorn/meshes/coupler/collision/COUPLER.stl; visual mesh filename=package://longhorn/meshes/coupler/visual/COUPLER.stl
- added link sia20d_arm_kinect; collision box size=0.36 0.28 0.22
- added link sia20d_arm_kinect_frame; collision box size=0.064 0.28 0.04; visual box size=0.064 0.28 0.04
- added link sia20d_arm_kinect_ir_link; visual sphere radius=0.0005
- added link sia20d_arm_kinect_ir_optical_frame
- added link sia20d_arm_kinect_keepout; collision box size=0.2 0.32 0.9
- added link sia20d_arm_kinect_rgb_link; visual sphere radius=0.0005
- added link sia20d_arm_kinect_rgb_optical_frame
- added link sia20d_arm_link_b; collision mesh filename=package://motoman_config/meshes/sia20d/collision/MOTOMAN_AX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; visual mesh filename=package://motoman_config/meshes/sia20d/visual/MOTOMAN_AXIS_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
- added link sia20d_arm_link_e; collision mesh filename=package://motoman_config/meshes/sia20d/collision/MOTOMAN_AX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; visual mesh filename=package://motoman_config/meshes/sia20d/visual/MOTOMAN_AXIS_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
- added link sia20d_arm_link_l; collision mesh filename=package://motoman_config/meshes/sia20d/collision/MOTOMAN_AX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; visual mesh filename=package://motoman_config/meshes/sia20d/visual/MOTOMAN_AXIS_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
- added link sia20d_arm_link_r; collision mesh filename=package://motoman_config/meshes/sia20d/collision/MOTOMAN_AX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; visual mesh filename=package://motoman_config/meshes/sia20d/visual/MOTOMAN_AXIS_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
- added link sia20d_arm_link_s; collision mesh filename=package://motoman_config/meshes/sia20d/collision/MOTOMAN_AX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; visual mesh filename=package://motoman_config/meshes/sia20d/visual/MOTOMAN_AXIS_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
- added link sia20d_arm_link_t; collision mesh filename=package://motoman_config/meshes/sia20d/collision/MOTOMAN_AX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; visual mesh filename=package://motoman_config/meshes/sia20d/visual/MOTOMAN_AXIS_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
- added link sia20d_arm_link_u; collision mesh filename=package://motoman_config/meshes/sia20d/collision/MOTOMAN_AX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; visual mesh filename=package://motoman_config/meshes/sia20d/visual/MOTOMAN_AXIS_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
- added link sia20d_arm_palm; collision box size=0.044 0.088 0.0946; visual box size=0.044 0.088 0.0946
Joints:
- removed joint sia20d_arm/joint_b
- removed joint sia20d_arm/joint_e
- removed joint sia20d_arm/joint_l
- removed joint sia20d_arm/joint_r
- removed joint sia20d_arm/joint_s
- removed joint sia20d_arm/joint_t
- removed joint sia20d_arm/joint_u
- removed joint sia20d_arm/kinect_frame_joint
- removed joint sia20d_arm/kinect_ir_joint
- removed joint sia20d_arm/kinect_ir_optical_frame_joint
- removed joint sia20d_arm/kinect_rgb_joint
- removed joint sia20d_arm/kinect_rgb_optical_frame_joint
- removed joint sia20d_arm/workcell_frame_to_kinect
- removed joint sia20d_arm/workcell_frame_to_kinect_keepout
- added joint joint_b: type revolute, parent sia20d_arm_link_r, child sia20d_arm_link_b, origin xyz=0 0 0 rpy=0 0 0, axis 0 -1 0, limit lower=-1.91 upper=1.91 effort=100 velocity=3.48
- added joint joint_e: type revolute, parent sia20d_arm_link_l, child sia20d_arm_link_e, origin xyz=0 0 0.49 rpy=0 0 0, axis 0 0 1, limit lower=-2.96 upper=2.96 effort=100 velocity=2.96
- added joint joint_l: type revolute, parent sia20d_arm_link_s, child sia20d_arm_link_l, origin xyz=0 0 0 rpy=0 0 0, axis 0 1 0, limit lower=-1.91 upper=1.91 effort=100 velocity=2.26
- added joint joint_r: type revolute, parent sia20d_arm_link_u, child sia20d_arm_link_r, origin xyz=0 0 0.420 rpy=0 0 0, axis 0 0 -1, limit lower=-3.1416 upper=3.1416 effort=100 velocity=3.48
- added joint joint_s: type revolute, parent sia20d_arm_base_link, child sia20d_arm_link_s, origin xyz=0 0 0.41 rpy=0 0 0, axis 0 0 1, limit lower=-3.1416 upper=3.1416 effort=100 velocity=2.26
- added joint joint_t: type revolute, parent sia20d_arm_link_b, child sia20d_arm_link_t, origin xyz=0 0 0.18 rpy=0 0 0, axis 0 0 -1, limit lower=-3.1416 upper=3.1416 effort=100 velocity=6.97
- added joint joint_u: type revolute, parent sia20d_arm_link_e, child sia20d_arm_link_u, origin xyz=0 0 0 rpy=0 0 0, axis 0 -1 0, limit lower=-2.26 upper=2.26 effort=100 velocity=2.96
- added joint sia20d_arm_kinect_frame_joint: type fixed, parent sia20d_arm_kinect, child sia20d_arm_kinect_frame, origin xyz=0 0 0 rpy=0 0 0
- added joint sia20d_arm_kinect_ir_joint: type fixed, parent sia20d_arm_kinect_frame, child sia20d_arm_kinect_ir_link, origin xyz=0 0 0 rpy=0 0 0
- added joint sia20d_arm_kinect_ir_optical_frame_joint: type fixed, parent sia20d_arm_kinect_ir_link, child sia20d_arm_kinect_ir_optical_frame, origin xyz=0 0 0 rpy=-1.57 0 -1.57
- added joint sia20d_arm_kinect_rgb_joint: type fixed, parent sia20d_arm_kinect_ir_link, child sia20d_arm_kinect_rgb_link, origin xyz=0 -0.03 0 rpy=0 0 0
- added joint sia20d_arm_kinect_rgb_optical_frame_joint: type fixed, parent sia20d_arm_kinect_rgb_link, child sia20d_arm_kinect_rgb_optical_frame, origin xyz=0 0 0 rpy=-1.57 0 -1.57
- added joint sia20d_arm_sia20d_arm_base_link_to_kinect: type fixed, parent sia20d_arm_base_link, child sia20d_arm_kinect, origin xyz=1.08 -0.72 0.82 rpy=0 0.5235 2.356
- added joint sia20d_arm_sia20d_arm_base_link_to_kinect_keepout: type fixed, parent sia20d_arm_base_link, child sia20d_arm_kinect_keepout, origin xyz=1.08 -0.72 0.45 rpy=0 0 2.356
- joint coupler-hand: child sia20d_arm/palm -> sia20d_arm_palm; parent sia20d_arm/coupler -> sia20d_arm_coupler
- joint sia20d_to_workcell: child sia20d_arm/base_link -> sia20d_arm_base_link
- joint tool-coupler: child sia20d_arm/coupler -> sia20d_arm_coupler; parent sia20d_arm/link_t -> sia20d_arm_link_t

File: mantis/mantis_config/urdf/mantis_sia20d_arm_workspace.xacro (robot description, xacro)
@@ -1,5 +1,5 @@
 <?xml version="1.0" ?>
 <robot name="mantis_sia20d" xmlns:xacro="http://ros.org/wiki/xacro">
-	<include filename="$(find motoman_config)/cfg/sia20d_mesh_macro.xacro"/>
+	<include filename="$(find mantis_config)/urdf/sia20d_mesh_macro.xacro"/>
 	<include filename="$(find mantis_config)/urdf/vacuum_gripper.xacro"/>
 	<include filename="$(find mantis_config)/urdf/vacuum_gripper_macro.xacro"/>
@@ -9,5 +9,6 @@
 	<xacro:property name="workcell_height" value="1"/>
 	<xacro:property name="vacuum_gripper_width" value="0.088"/>
-	<xacro:property name="arm1_prefix" value="sia20d_arm/"/>
+	<xacro:property name="arm1_prefix" value="sia20d_arm_"/>
+	<!--xacro:property name="arm1_prefix" value=""/-->
 	<xacro:property name="arm1_name" value="sia20d"/>
 	<!-- instantiating workcell definitions -->
@@ -15,6 +16,8 @@
 	<!-- end of workcell definitions -->
 	<!-- instantiating sensor definitions -->
-	<xacro:sensor_definitions prefix="${arm1_prefix}" parent_link="workcell_frame"
-		x_val="1.20" y_val="0" z_val="0.4" pitch="0.5235" yaw="3.147"/>
+	<!--xacro:sensor_definitions prefix="${arm1_prefix}" parent_link="workcell_frame"
+		x_val="1.20" y_val="0" z_val="0.4" pitch="0.5235" yaw="3.147"/-->
+	<xacro:sensor_definitions prefix="${arm1_prefix}" parent_link="${arm1_prefix}base_link"
+		x_val="1.08" y_val="-0.72" z_val="0.82" pitch="0.5235" yaw="2.356"/>
 	<!-- end of sensor definitions -->
 	<!-- instantiating arm and gripper -->
