Commit message: launch files for sia20d navigation updated
git-svn-id: http://swri-ros-pkg.googlecode.com/svn/trunk@726 076cdf4d-ed99-c8c1-5d01-9bc0d27e81bd

File: mantis/mantis_config/urdf/mantis_ur5.urdf (robot description, URDF)
Before this commit: robot mantis_ur5, 27 links, 26 joints
Links:
- removed link ur5_arm/base_link
- removed link ur5_arm/ee_link
- removed link ur5_arm/forearm_link
- removed link ur5_arm/gripper_body
- removed link ur5_arm/gripper_frame
- removed link ur5_arm/kinect
- removed link ur5_arm/kinect_frame
- removed link ur5_arm/kinect_ir_link
- removed link ur5_arm/kinect_ir_optical_frame
- removed link ur5_arm/kinect_keepout
- removed link ur5_arm/kinect_rgb_link
- removed link ur5_arm/kinect_rgb_optical_frame
- removed link ur5_arm/shoulder_link
- removed link ur5_arm/tcp_frame
- removed link ur5_arm/upper_arm_link
- removed link ur5_arm/wrist_1_link
- removed link ur5_arm/wrist_2_link
- removed link ur5_arm/wrist_3_link
- added link ur5_arm_base_link, mass 4.0; visual mesh filename=package://ur5_description/meshes/Base.dae
- added link ur5_arm_ee_link
- added link ur5_arm_forearm_link, mass 2.275; collision cylinder length=0.39225 radius=0.04; visual mesh filename=package://ur5_description/meshes/Forearm.dae
- added link ur5_arm_gripper_body; collision box size=0.044 0.088 0.0946; visual box size=0.044 0.088 0.0946
- added link ur5_arm_gripper_frame
- added link ur5_arm_kinect; collision box size=0.36 0.28 0.22
- added link ur5_arm_kinect_frame; collision box size=0.064 0.28 0.04; visual box size=0.064 0.28 0.04
- added link ur5_arm_kinect_ir_link; visual sphere radius=0.0005
- added link ur5_arm_kinect_ir_optical_frame
- added link ur5_arm_kinect_keepout; collision box size=0.2 0.32 0.48
- added link ur5_arm_kinect_rgb_link; visual sphere radius=0.0005
- added link ur5_arm_kinect_rgb_optical_frame
- added link ur5_arm_shoulder_link, mass 3.7; collision cylinder length=0.16 radius=0.06; visual mesh filename=package://ur5_description/meshes/Shoulder.dae
- added link ur5_arm_tcp_frame
- added link ur5_arm_upper_arm_link, mass 8.393; collision cylinder length=0.425 radius=0.054; visual mesh filename=package://ur5_description/meshes/UpperArm.dae
- added link ur5_arm_wrist_1_link, mass 1.219; collision cylinder length=0.1488 radius=0.045; visual mesh filename=package://ur5_description/meshes/Wrist1.dae
- added link ur5_arm_wrist_2_link, mass 1.219; collision cylinder length=0.15144 radius=0.045; visual mesh filename=package://ur5_description/meshes/Wrist2.dae
- added link ur5_arm_wrist_3_link, mass 0.1879; collision cylinder length=0.135795 radius=0.045; visual mesh filename=package://ur5_description/meshes/Wrist3.dae
Joints:
- removed joint ur5_arm/ee_fixed_joint
- removed joint ur5_arm/elbow_joint
- removed joint ur5_arm/gripper_to_palm
- removed joint ur5_arm/gripper_to_tcp
- removed joint ur5_arm/kinect_frame_joint
- removed joint ur5_arm/kinect_ir_joint
- removed joint ur5_arm/kinect_ir_optical_frame_joint
- removed joint ur5_arm/kinect_rgb_joint
- removed joint ur5_arm/kinect_rgb_optical_frame_joint
- removed joint ur5_arm/shoulder_lift_joint
- removed joint ur5_arm/shoulder_pan_joint
- removed joint ur5_arm/workcell_frame_to_kinect
- removed joint ur5_arm/workcell_frame_to_kinect_keepout
- removed joint ur5_arm/wrist_1_joint
- removed joint ur5_arm/wrist_2_joint
- removed joint ur5_arm/wrist_3_joint
- added joint ur5_arm_ee_fixed_joint: type fixed, parent ur5_arm_wrist_3_link, child ur5_arm_ee_link, origin xyz=0.0 0.0823 0.0 rpy=0.0 0.0 1.570796325
- added joint ur5_arm_elbow_joint: type revolute, parent ur5_arm_upper_arm_link, child ur5_arm_forearm_link, origin xyz=0.0 -0.1197 0.425 rpy=0.0 0.0 0.0, axis 0.0 1.0 0.0, limit lower=-6.2831853 upper=6.2831853 effort=10.0 velocity=3.14159265
- added joint ur5_arm_gripper_to_palm: type fixed, parent ur5_arm_gripper_frame, child ur5_arm_gripper_body, origin xyz=0 0 0.0473 rpy=0 0 0
- added joint ur5_arm_gripper_to_tcp: type fixed, parent ur5_arm_gripper_frame, child ur5_arm_tcp_frame, origin xyz=0.022 0 0.0946 rpy=0 0 0
- added joint ur5_arm_kinect_frame_joint: type fixed, parent ur5_arm_kinect, child ur5_arm_kinect_frame, origin xyz=0 0 0 rpy=0 0 0
- added joint ur5_arm_kinect_ir_joint: type fixed, parent ur5_arm_kinect_frame, child ur5_arm_kinect_ir_link, origin xyz=0 0 0 rpy=0 0 0
- added joint ur5_arm_kinect_ir_optical_frame_joint: type fixed, parent ur5_arm_kinect_ir_link, child ur5_arm_kinect_ir_optical_frame, origin xyz=0 0 0 rpy=-1.57 0 -1.57
- added joint ur5_arm_kinect_rgb_joint: type fixed, parent ur5_arm_kinect_ir_link, child ur5_arm_kinect_rgb_link, origin xyz=0 -0.03 0 rpy=0 0 0
- added joint ur5_arm_kinect_rgb_optical_frame_joint: type fixed, parent ur5_arm_kinect_rgb_link, child ur5_arm_kinect_rgb_optical_frame, origin xyz=0 0 0 rpy=-1.57 0 -1.57
- added joint ur5_arm_shoulder_lift_joint: type revolute, parent ur5_arm_shoulder_link, child ur5_arm_upper_arm_link, origin xyz=0.0 0.13585 0.0 rpy=0.0 1.570796325 0.0, axis 0.0 1.0 0.0, limit lower=-6.2831853 upper=6.2831853 effort=10.0 velocity=3.14159265
- added joint ur5_arm_shoulder_pan_joint: type revolute, parent ur5_arm_base_link, child ur5_arm_shoulder_link, origin xyz=0.0 0.0 0.089159 rpy=0.0 0.0 0.0, axis 0.0 0.0 1.0, limit lower=-6.2831853 upper=6.2831853 effort=10.0 velocity=3.14159265
- added joint ur5_arm_workcell_frame_to_kinect: type fixed, parent workcell_frame, child ur5_arm_kinect, origin xyz=-1.2 0 0.4 rpy=0 0.5235 0
- added joint ur5_arm_workcell_frame_to_kinect_keepout: type fixed, parent workcell_frame, child ur5_arm_kinect_keepout, origin xyz=-1.2 0 0.24 rpy=0 0 0
- added joint ur5_arm_wrist_1_joint: type revolute, parent ur5_arm_forearm_link, child ur5_arm_wrist_1_link, origin xyz=0.0 0.0 0.39225 rpy=0.0 1.570796325 0.0, axis 0.0 1.0 0.0, limit lower=-6.2831853 upper=6.2831853 effort=10.0 velocity=3.14159265
- added joint ur5_arm_wrist_2_joint: type revolute, parent ur5_arm_wrist_1_link, child ur5_arm_wrist_2_link, origin xyz=0.0 0.093 0.0 rpy=0.0 0.0 0.0, axis 0.0 0.0 1.0, limit lower=-6.2831853 upper=6.2831853 effort=10.0 velocity=3.14159265
- added joint ur5_arm_wrist_3_joint: type revolute, parent ur5_arm_wrist_2_link, child ur5_arm_wrist_3_link, origin xyz=0.0 0.0 0.09465 rpy=0.0 0.0 0.0, axis 0.0 1.0 0.0, limit lower=-6.2831853 upper=6.2831853 effort=10.0 velocity=3.14159265
- joint ur5_to_gripper: child ur5_arm/gripper_frame -> ur5_arm_gripper_frame; parent ur5_arm/ee_link -> ur5_arm_ee_link
- joint ur5_to_stand: child ur5_arm/base_link -> ur5_arm_base_link

File: mantis/mantis_config/urdf/mantis_ur5_arm_workspace.xacro (robot description, xacro)
@@ -9,5 +9,5 @@
 	<xacro:property name="workcell_height" value="1"/>
 	<xacro:property name="vacuum_gripper_width" value="0.088"/>
-	<xacro:property name="arm2_prefix" value="ur5_arm/"/>
+	<xacro:property name="arm2_prefix" value="ur5_arm_"/>
 	<xacro:property name="arm2_name" value="ur5"/>
 	<!-- instantiating arm and gripper -->
